File: modules/Oddities_RevA_10Mar2011.kicad_pcb (KiCad board)
At the start: 2 copper layers, 16 parts

Commit message: TO-78 stuff added.
Other:
- board text added: "Oddities_RevA_10Mar2011.mod"
- board text added: "You can use an empty modul if you want some parts at the schematic, but not at the layout. Netties are some "devices" with two and more separated pads and a connection between them. They are used to tie different ground system as signal ground and digital grond together at only one point."
- board text removed: "Footprint-Symbols_RevD_28Aug2012.mod"
Changed lines of the file:
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@@
     (links 0)
     (no_connects 0)
-    (area -16.90696 21.436 274.02378 197.1694)
+    (area -16.90696 15.555699 274.02378 197.1694)
     (thickness 1.6002)
-    (drawings 7)
+    (drawings 8)
     (tracks 0)
     (zones 0)
@@
     )
   )
+  (gr_text "You can use an empty modul if you want some parts at the\nschematic, but not at the layout. \n\nNetties are some \"devices\" with two and more separated pads and a\nconnection between them. They are used to tie different ground system\nas signal ground and digital grond together at only one point." (at 64 37.5) (layer F.SilkS)
+    (effects (font (size 2.032 1.524) (thickness 0.3048)))
+  )
   (gr_text http://creativecommons.org/ (at 98 192.5) (layer F.SilkS)
     (effects (font (size 3 3) (thickness 0.6)))
@@
     (effects (font (size 4.0005 4.0005) (thickness 0.59944)))
   )
-  (gr_text "Footprint-Symbols_RevD_28Aug2012.mod\n" (at 117 152.5) (layer F.SilkS)
+  (gr_text "Oddities_RevA_10Mar2011.mod\n" (at 117 152.5) (layer F.SilkS)
     (effects (font (size 4.0005 4.0005) (thickness 0.59944)))
   )
