File: modules/EuroBoardoutline_RevC_Part3.kicad_pcb (KiCad board)
At the start: 2 copper layers, 100 x 40 mm, 7 parts

Commit message: EuroBoardOutline shifted to revision C. forgotten SMD capacitors addet.
Parts:
- removed the Outl at (36.0, 61.0)
- removed the Outl at (36.5, 120.5)
- removed the Outl at (166.5, 69.0)
- removed the Outl at (166.5, 133.5)
- added Outl: EuroBoard_achtel_Type-I_40mmX50mm_holes, EuroBoard_achtel_Type-I_40mmX50mm_holes, F.Cu at (165.0, 70.5)
- added Outl: EuroBoard_achtel_Type-I_40mmX50mm, EuroBoard_achtel_Type-I_40mmX50mm, F.Cu at (40.5, 72.0)
- added Outl: EuroBoard_halb_Type-II_160mmX50mm, EuroBoard_halb_Type-II_160mmX50mm, F.Cu at (61.0, 133.5)
Other:
- board size 100 x 40 mm -> 160 x 50 mm
- board text added: "Author: Bernd Wiebus / Uedem / Germany / 07 Jun 2013"
- board text added: "EuroBoardoutline_RevC.mod"
- board text removed: "Author: Bernd Wiebus / Uedem / Germany / 04 Jun 2013"
- board text removed: "EuroBoardoutline_RevB.mod"
Changed lines of the file:
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@@
     (links 0)
     (no_connects 0)
-    (area -16.90696 13.9963 275.720423 197.1694)
+    (area -16.90696 15.4963 284.55359 197.1694)
     (thickness 1.6002)
     (drawings 7)
     (tracks 0)
     (zones 0)
-    (modules 7)
+    (modules 6)
     (nets 1)
   )
@@
     (mod_text_size 1.524 1.524)
     (mod_text_width 0.3048)
-    (pad_size 1.524 1.524)
-    (pad_drill 0.8128)
+    (pad_size 3.50012 3.50012)
+    (pad_drill 3.50012)
     (pad_to_mask_clearance 0.254)
     (aux_axis_origin 0 0)
@@
     (uvia_drill 0.127)
     (add_net "")
+  )
+  (module EuroBoard_achtel_Type-I_40mmX50mm_holes (layer Vorderseite)
+    (at 165 70.5)
+    (descr "Outline, Eurocard 1/8, Type I,  40x50mm, with holes 3,5mm,")
+    (tags "Outline, Eurocard 1/8, Type I, 40x50mm, with holes 3,5mm,")
+    (fp_text reference Outl (at 19.99996 -52.99964) (layer F.SilkS)
+      (effects (font (size 2.99974 2.99974) (thickness 0.50038)))
+    )
+    (fp_text value EuroBoard_achtel_Type-I_40mmX50mm_holes (at 54 5) (layer F.SilkS)
+      (effects (font (size 3.00228 3.00228) (thickness 0.50038)))
+    )
+    (fp_line (start 0 0) (end 39.99992 0) (layer Edge.Cuts) (width 0.381))
+    (fp_line (start 39.99992 0) (end 39.99992 -49.9999) (layer Edge.Cuts) (width 0.381))
+    (fp_line (start 39.99992 -49.9999) (end 0 -49.9999) (layer Edge.Cuts) (width 0.381))
+    (fp_line (start 0 -49.9999) (end 0 0) (layer Edge.Cuts) (width 0.381))
+    (pad "" np_thru_hole circle (at 5.00126 -5.00126) (size 3.50012 3.50012) (drill 3.50012)
+      (layers *.Cu *.Mask F.SilkS)
+    )
+    (pad "" np_thru_hole circle (at 5.00126 -45.00118) (size 3.50012 3.50012) (drill 3.50012)
+      (layers *.Cu *.Mask F.SilkS)
+    )
+    (pad "" np_thru_hole circle (at 35.0012 -45.00118) (size 3.50012 3.50012) (drill 3.50012)
+      (layers *.Cu *.Mask F.SilkS)
+    )
+    (pad "" np_thru_hole circle (at 35.0012 -5.00126) (size 3.50012 3.50012) (drill 3.50012)
+      (layers *.Cu *.Mask F.SilkS)
+    )
   )
   (module Gauge_100mm_Type2_SilkScreenTop_RevA_Date22Jun2010 (layer Vorderseite)
@@
     (fp_circle (center 0 0) (end 5.588 0) (layer F.SilkS) (width 0.381))
   )
-  (module EuroBoard_viertel_Type-II_100mmX40mm (layer Vorderseite)
-    (at 36 61)
-    (descr "Outline, Eurocard 1/4, Type I, 100x40mm,")
-    (tags "Outline, Eurocard 1/4, Type II, 100x40mm,")
-    (fp_text reference Outl (at 51.99888 -44.00042) (layer F.SilkS)
+  (module EuroBoard_achtel_Type-I_40mmX50mm (layer Vorderseite)
+    (at 40.5 72)
+    (descr "Outline, Eurocard 1/8, Type I,  40x50mm,")
+    (tags "Outline, Eurocard 1/8, Type I, 40x50mm,")
+    (fp_text reference Outl (at 19.99996 -52.99964) (layer F.SilkS)
       (effects (font (size 2.99974 2.99974) (thickness 0.50038)))
     )
-    (fp_text value EuroBoard_viertel_Type-II_100mmX40mm (at 51.00066 7.00024) (layer F.SilkS)
+    (fp_text value EuroBoard_achtel_Type-I_40mmX50mm (at 45.5 6) (layer F.SilkS)
       (effects (font (size 3.00228 3.00228) (thickness 0.50038)))
     )
-    (fp_line (start 0 0) (end 99.9998 0) (layer Edge.Cuts) (width 0.381))
-    (fp_line (start 99.9998 0) (end 99.9998 -39.99992) (layer Edge.Cuts) (width 0.381))
-    (fp_line (start 99.9998 -39.99992) (end 0 -39.99992) (layer Edge.Cuts) (width 0.381))
-    (fp_line (start 0 -39.99992) (end 0 0) (layer Edge.Cuts) (width 0.381))
-  )
-  (module EuroBoard_viertel_Type-II_100mmX40mm_holes (layer Vorderseite)
-    (at 36.5 120.5)
-    (descr "Outline, Eurocard 1/4, Type I, 100x40mm, with holes 3,5mm,")
-    (tags "Outline, Eurocard 1/4, Type II, 100x40mm, with holes 3,5mm,")
-    (fp_text reference Outl (at 51.99888 -44.00042) (layer F.SilkS)
+    (fp_line (start 0 0) (end 39.99992 0) (layer Edge.Cuts) (width 0.381))
+    (fp_line (start 39.99992 0) (end 39.99992 -49.9999) (layer Edge.Cuts) (width 0.381))
+    (fp_line (start 39.99992 -49.9999) (end 0 -49.9999) (layer Edge.Cuts) (width 0.381))
+    (fp_line (start 0 -49.9999) (end 0 0) (layer Edge.Cuts) (width 0.381))
+  )
+  (module EuroBoard_halb_Type-II_160mmX50mm (layer Vorderseite)
+    (at 61 133.5)
+    (descr "Outline, Eurocard 1/2, Type II, 160x50mm,")
+    (tags "Outline, Eurocard 1/2, Type II, 160x50mm,")
+    (path EuroBoard-halb-100mmX80mm)
+    (fp_text reference Outl (at 67.5 -35) (layer F.SilkS)
       (effects (font (size 2.99974 2.99974) (thickness 0.50038)))
     )
-    (fp_text value EuroBoard_viertel_Type-II_100mmX40mm_holes (at 51.00066 7.00024) (layer F.SilkS)
+    (fp_text value EuroBoard_halb_Type-II_160mmX50mm (at 73 -6.5) (layer F.SilkS)
       (effects (font (size 3.00228 3.00228) (thickness 0.50038)))
     )
-    (fp_line (start 0 0) (end 99.9998 0) (layer Edge.Cuts) (width 0.381))
-    (fp_line (start 99.9998 0) (end 99.9998 -39.99992) (layer Edge.Cuts) (width 0.381))
-    (fp_line (start 99.9998 -39.99992) (end 0 -39.99992) (layer Edge.Cuts) (width 0.381))
-    (fp_line (start 0 -39.99992) (end 0 0) (layer Edge.Cuts) (width 0.381))
-    (pad 1 thru_hole circle (at 5.00126 -5.00126) (size 3.50012 3.50012) (drill 3.50012)
-      (layers *.Cu *.Mask F.SilkS)
-    )
-    (pad 2 thru_hole circle (at 5.00126 -35.0012) (size 3.50012 3.50012) (drill 3.50012)
-      (layers *.Cu *.Mask F.SilkS)
-    )
-    (pad 3 thru_hole circle (at 95.00108 -35.0012) (size 3.50012 3.50012) (drill 3.50012)
-      (layers *.Cu *.Mask F.SilkS)
-    )
-    (pad 4 thru_hole circle (at 95.00108 -5.00126) (size 3.50012 3.50012) (drill 3.50012)
-      (layers *.Cu *.Mask F.SilkS)
-    )
-  )
-  (module EuroBoard_viertel_Type-I_80mmX50mm (layer Vorderseite)
-    (at 166.5 69)
-    (descr "Outline, Eurocard 1/4, Type I,  80x50mm,")
-    (tags "Outline, Eurocard 1/4, Type I, 80x50mm,")
-    (fp_text reference Outl (at 41.00068 -52.99964) (layer F.SilkS)
-      (effects (font (size 2.99974 2.99974) (thickness 0.50038)))
-    )
-    (fp_text value EuroBoard_viertel_Type-I_80mmX50mm (at 41.9989 5.99948) (layer F.SilkS)
-      (effects (font (size 3.00228 3.00228) (thickness 0.50038)))
-    )
-    (fp_line (start 0 0) (end 0 -49.9999) (layer Edge.Cuts) (width 0.381))
-    (fp_line (start 0 -49.9999) (end 79.99984 -49.9999) (layer Edge.Cuts) (width 0.381))
-    (fp_line (start 79.99984 -49.9999) (end 79.99984 0) (layer Edge.Cuts) (width 0.381))
-    (fp_line (start 79.99984 0) (end 0 0) (layer Edge.Cuts) (width 0.381))
-  )
-  (module EuroBoard_viertel_Type-I_80mmX50mm_holes (layer Vorderseite)
-    (at 166.5 133.5)
-    (descr "Outline, Eurocard 1/4, Type I,  80x50mm, with holes 3,5mm,")
-    (tags "Outline, Eurocard 1/4, Type I, 80x50mm, with holes 3,5mm,")
-    (fp_text reference Outl (at 41.00068 -54.0004) (layer F.SilkS)
-      (effects (font (size 2.99974 2.99974) (thickness 0.50038)))
-    )
-    (fp_text value EuroBoard_viertel_Type-I_80mmX50mm_holes (at 41.9989 5.00126) (layer F.SilkS)
-      (effects (font (size 3.00228 3.00228) (thickness 0.50038)))
-    )
-    (fp_line (start 0 0) (end 0 -49.9999) (layer Edge.Cuts) (width 0.381))
-    (fp_line (start 0 -49.9999) (end 79.99984 -49.9999) (layer Edge.Cuts) (width 0.381))
-    (fp_line (start 79.99984 -49.9999) (end 79.99984 0) (layer Edge.Cuts) (width 0.381))
-    (fp_line (start 79.99984 0) (end 0 0) (layer Edge.Cuts) (width 0.381))
-    (pad 1 thru_hole circle (at 5.00126 -5.00126) (size 3.50012 3.50012) (drill 3.50012)
-      (layers *.Cu *.Mask F.SilkS)
-    )
-    (pad 2 thru_hole circle (at 5.00126 -45.00118) (size 3.50012 3.50012) (drill 3.50012)
-      (layers *.Cu *.Mask F.SilkS)
-    )
-    (pad 3 thru_hole circle (at 75.00112 -45.00118) (size 3.50012 3.50012) (drill 3.50012)
-      (layers *.Cu *.Mask F.SilkS)
-    )
-    (pad 4 thru_hole circle (at 75.00112 -5.00126) (size 3.50012 3.50012) (drill 3.50012)
-      (layers *.Cu *.Mask F.SilkS)
-    )
+    (fp_line (start 0 0) (end 159.99968 0) (layer Edge.Cuts) (width 0.381))
+    (fp_line (start 159.99968 0) (end 159.99968 -49.9999) (layer Edge.Cuts) (width 0.381))
+    (fp_line (start 159.99968 -49.9999) (end 0 -49.9999) (layer Edge.Cuts) (width 0.381))
+    (fp_line (start 0 -49.9999) (end 0 0) (layer Edge.Cuts) (width 0.381))
   )
   (gr_text http://creativecommons.org/ (at 98 192.5) (layer F.SilkS)
@@
     (effects (font (size 4.0005 4.0005) (thickness 0.59944)))
   )
-  (gr_text "Author: Bernd Wiebus / Uedem / Germany / 04 Jun 2013" (at 114.50012 172.24958) (layer F.SilkS)
+  (gr_text "Author: Bernd Wiebus / Uedem / Germany / 07 Jun 2013" (at 114.50012 172.24958) (layer F.SilkS)
     (effects (font (size 4.0005 4.0005) (thickness 0.59944)))
   )
-  (gr_text EuroBoardoutline_RevB.mod (at 114.00028 165.9989) (layer F.SilkS)
+  (gr_text EuroBoardoutline_RevC.mod (at 114.00028 165.9989) (layer F.SilkS)
     (effects (font (size 4.0005 4.0005) (thickness 0.59944)))
   )
