File: modules/EuroBoardoutline_RevC_Part4.kicad_pcb (KiCad board)
At the start: 2 copper layers, 160 x 50 mm, 6 parts

Commit message: EuroBoardOutline shifted to revision C. forgotten SMD capacitors addet.
Parts:
- removed the Outl at (40.5, 72.0)
- removed the Outl at (165.0, 70.5)
- removed the Outl at (61.0, 138.0)
- added Outl: EuroBoard_sechzehntel_Type-I_40mmX25mm, EuroBoard_sechzehntel_Type-I_40mmX25mm, F.Cu at (68.5, 51.0)
- added Outl: EuroBoard_sechzehntel_Type-I_40mmX25mm_holes, EuroBoard_sechzehntel_Type-I_40mmX25mm_holes, F.Cu at (199.0, 51.0)
- added Outl: EuroBoard_halb_Type-II_160mmX50mm_holes, EuroBoard_halb_Type-II_160mmX50mm_holes, F.Cu at (68.5, 124.5)
Other:
- board text added: "Author: Bernd Wiebus / Uedem / Germany / 07 Jun 2013"
- board text added: "EuroBoardoutline_RevC.mod"
- board text removed: "Author: Bernd Wiebus / Uedem / Germany / 04 Jun 2013"
- board text removed: "EuroBoardoutline_RevB.mod"
Changed lines of the file:
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@@
     (links 0)
     (no_connects 0)
-    (area -16.90696 15.4963 284.55359 197.1694)
+    (area -16.90696 18.49676 289.893216 197.1694)
     (thickness 1.6002)
     (drawings 7)
@@
     (fp_circle (center 0 0) (end 5.588 0) (layer F.SilkS) (width 0.381))
   )
-  (module EuroBoard_achtel_Type-I_40mmX50mm (layer Vorderseite)
-    (at 40.5 72)
-    (descr "Outline, Eurocard 1/8, Type I,  40x50mm,")
-    (tags "Outline, Eurocard 1/8, Type I, 40x50mm,")
-    (fp_text reference Outl (at 19.99996 -52.99964) (layer F.SilkS)
+  (module EuroBoard_sechzehntel_Type-I_40mmX25mm (layer Vorderseite)
+    (at 68.5 51)
+    (descr "Outline, Eurocard 1/16, Type I,  40x25mm,")
+    (tags "Outline, Eurocard 1/16, Type I, 40x25mm,")
+    (fp_text reference Outl (at 19.99996 -28.99918) (layer F.SilkS)
       (effects (font (size 2.99974 2.99974) (thickness 0.50038)))
     )
-    (fp_text value EuroBoard_achtel_Type-I_40mmX50mm (at 45.5 6) (layer F.SilkS)
+    (fp_text value EuroBoard_sechzehntel_Type-I_40mmX25mm (at 19.99996 5.00126) (layer F.SilkS)
       (effects (font (size 3.00228 3.00228) (thickness 0.50038)))
     )
+    (fp_line (start 39.99992 0) (end 39.99992 -25.00122) (layer Edge.Cuts) (width 0.381))
+    (fp_line (start 39.99992 -25.00122) (end 0 -25.00122) (layer Edge.Cuts) (width 0.381))
+    (fp_line (start 0 -25.00122) (end 0 0) (layer Edge.Cuts) (width 0.381))
     (fp_line (start 0 0) (end 39.99992 0) (layer Edge.Cuts) (width 0.381))
-    (fp_line (start 39.99992 0) (end 39.99992 -49.9999) (layer Edge.Cuts) (width 0.381))
-    (fp_line (start 39.99992 -49.9999) (end 0 -49.9999) (layer Edge.Cuts) (width 0.381))
-    (fp_line (start 0 -49.9999) (end 0 0) (layer Edge.Cuts) (width 0.381))
-  )
-  (module EuroBoard_achtel_Type-I_40mmX50mm_holes (layer Vorderseite)
-    (at 165 70.5)
-    (descr "Outline, Eurocard 1/8, Type I,  40x50mm, with holes 3,5mm,")
-    (tags "Outline, Eurocard 1/8, Type I, 40x50mm, with holes 3,5mm,")
-    (fp_text reference Outl (at 19.99996 -52.99964) (layer F.SilkS)
+  )
+  (module EuroBoard_sechzehntel_Type-I_40mmX25mm_holes (layer Vorderseite)
+    (at 199 51)
+    (descr "Outline, Eurocard 1/16, Type I,  40x25mm, with holes 3,5mm,")
+    (tags "Outline, Eurocard 1/16, Type I, 40x25mm, with holes 3,5mm,")
+    (fp_text reference Outl (at 19.99996 -28.99918) (layer F.SilkS)
       (effects (font (size 2.99974 2.99974) (thickness 0.50038)))
     )
-    (fp_text value EuroBoard_achtel_Type-I_40mmX50mm_holes (at 54 5) (layer F.SilkS)
+    (fp_text value EuroBoard_sechzehntel_Type-I_40mmX25mm_holes (at 19.99996 5.00126) (layer F.SilkS)
       (effects (font (size 3.00228 3.00228) (thickness 0.50038)))
     )
+    (fp_line (start 39.99992 0) (end 39.99992 -25.00122) (layer Edge.Cuts) (width 0.381))
+    (fp_line (start 39.99992 -25.00122) (end 0 -25.00122) (layer Edge.Cuts) (width 0.381))
+    (fp_line (start 0 -25.00122) (end 0 0) (layer Edge.Cuts) (width 0.381))
     (fp_line (start 0 0) (end 39.99992 0) (layer Edge.Cuts) (width 0.381))
-    (fp_line (start 39.99992 0) (end 39.99992 -49.9999) (layer Edge.Cuts) (width 0.381))
-    (fp_line (start 39.99992 -49.9999) (end 0 -49.9999) (layer Edge.Cuts) (width 0.381))
-    (fp_line (start 0 -49.9999) (end 0 0) (layer Edge.Cuts) (width 0.381))
-    (pad 1 thru_hole circle (at 5.00126 -5.00126) (size 3.50012 3.50012) (drill 3.50012)
+    (pad "" np_thru_hole circle (at 5.00126 -12.49934) (size 3.50012 3.50012) (drill 3.50012)
       (layers *.Cu *.Mask F.SilkS)
     )
-    (pad 2 thru_hole circle (at 5.00126 -45.00118) (size 3.50012 3.50012) (drill 3.50012)
+    (pad "" np_thru_hole circle (at 34.50082 -12.49934) (size 3.50012 3.50012) (drill 3.50012)
       (layers *.Cu *.Mask F.SilkS)
     )
-    (pad 3 thru_hole circle (at 35.0012 -45.00118) (size 3.50012 3.50012) (drill 3.50012)
-      (layers *.Cu *.Mask F.SilkS)
-    )
-    (pad 4 thru_hole circle (at 35.0012 -5.00126) (size 3.50012 3.50012) (drill 3.50012)
-      (layers *.Cu *.Mask F.SilkS)
-    )
-  )
-  (module EuroBoard_halb_Type-II_160mmX50mm (layer Vorderseite)
-    (at 61 138)
-    (descr "Outline, Eurocard 1/2, Type II, 160x50mm,")
-    (tags "Outline, Eurocard 1/2, Type II, 160x50mm,")
+  )
+  (module EuroBoard_halb_Type-II_160mmX50mm_holes (layer Vorderseite)
+    (at 68.5 124.5)
+    (descr "Outline, Eurocard 1/2, Type II, 160x50mm, with holes 3,5mm,")
+    (tags "Outline, Eurocard 1/2, Type II, 160x50mm, with holes 3,5mm,")
     (path EuroBoard-halb-100mmX80mm)
-    (fp_text reference Outl (at 67.5 -35) (layer F.SilkS)
+    (fp_text reference Outl (at 77.0001 -54.0004) (layer F.SilkS)
       (effects (font (size 2.99974 2.99974) (thickness 0.50038)))
     )
-    (fp_text value EuroBoard_halb_Type-II_160mmX50mm (at 73 -6.5) (layer F.SilkS)
+    (fp_text value EuroBoard_halb_Type-II_160mmX50mm_holes (at 78.00086 5.99948) (layer F.SilkS)
       (effects (font (size 3.00228 3.00228) (thickness 0.50038)))
     )
@@
     (fp_line (start 159.99968 -49.9999) (end 0 -49.9999) (layer Edge.Cuts) (width 0.381))
     (fp_line (start 0 -49.9999) (end 0 0) (layer Edge.Cuts) (width 0.381))
+    (pad "" np_thru_hole circle (at 5.00126 -5.00126) (size 3.50012 3.50012) (drill 3.50012)
+      (layers *.Cu *.Mask F.SilkS)
+    )
+    (pad "" np_thru_hole circle (at 5.00126 -45.00118) (size 3.50012 3.50012) (drill 3.50012)
+      (layers *.Cu *.Mask F.SilkS)
+    )
+    (pad "" np_thru_hole circle (at 155.00096 -45.00118) (size 3.50012 3.50012) (drill 3.50012)
+      (layers *.Cu *.Mask F.SilkS)
+    )
+    (pad "" np_thru_hole circle (at 155.00096 -5.00126) (size 3.50012 3.50012) (drill 3.50012)
+      (layers *.Cu *.Mask F.SilkS)
+    )
   )
   (gr_text http://creativecommons.org/ (at 98 192.5) (layer F.SilkS)
@@
     (effects (font (size 4.0005 4.0005) (thickness 0.59944)))
   )
-  (gr_text "Author: Bernd Wiebus / Uedem / Germany / 04 Jun 2013" (at 114.50012 172.24958) (layer F.SilkS)
+  (gr_text "Author: Bernd Wiebus / Uedem / Germany / 07 Jun 2013" (at 114.50012 172.24958) (layer F.SilkS)
     (effects (font (size 4.0005 4.0005) (thickness 0.59944)))
   )
-  (gr_text EuroBoardoutline_RevB.mod (at 114.00028 165.9989) (layer F.SilkS)
+  (gr_text EuroBoardoutline_RevC.mod (at 114.00028 165.9989) (layer F.SilkS)
     (effects (font (size 4.0005 4.0005) (thickness 0.59944)))
   )
