File: modules/EuroBoardoutline_RevC_Part6.kicad_pcb (KiCad board)
At the start: 2 copper layers, 160 x 100 mm, 5 parts

Commit message: EuroBoardOutline shifted to revision C. forgotten SMD capacitors addet.
Parts:
- removed the Outl at (48.0, 129.0)
- removed the Outl at (255.5, 119.0)
- added Outl: EuroBoard_viertel_Type-III_160mmX25mm, EuroBoard_viertel_Type-III_160mmX25mm, F.Cu at (73.0, 42.0)
- added Outl: EuroBoard_viertel_Type-II_100mmX40mm, EuroBoard_viertel_Type-II_100mmX40mm, F.Cu at (58.0, 125.0)
- added Outl: EuroBoard_viertel_Type-III_160mmX25mm_holes, EuroBoard_viertel_Type-III_160mmX25mm_holes, F.Cu at (73.0, 75.0)
- added Outl: EuroBoard_viertel_Type-II_100mmX40mm_holes, EuroBoard_viertel_Type-II_100mmX40mm_holes, F.Cu at (172.5, 125.0)
Other:
- board size 160 x 100 mm -> 160 x 25 mm
- board text added: "Author: Bernd Wiebus / Uedem / Germany / 07 Jun 2013"
- board text added: "EuroBoardoutline_RevC.mod"
- board text removed: "Author: Bernd Wiebus / Uedem / Germany / 04 Jun 2013"
- board text removed: "EuroBoardoutline_RevB.mod"
Changed lines of the file:
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@@
     (links 0)
     (no_connects 0)
-    (area -16.90696 9.779577 274.02378 197.1694)
+    (area -16.90696 16.554279 301.05739 197.1694)
     (thickness 1.6002)
     (drawings 7)
     (tracks 0)
     (zones 0)
-    (modules 5)
+    (modules 7)
     (nets 1)
   )
@@
     (fp_circle (center 0 0) (end 5.588 0) (layer F.SilkS) (width 0.381))
   )
-  (module EuroBoard160mmX100mm_holes (layer Vorderseite)
-    (at 48 129)
-    (descr "Outline, Eurocard, 100x160mm, with holes 3,5mm,")
-    (tags "Outline, Eurocard, 100x160mm, with holes 3,5mm,")
-    (fp_text reference Outl (at 78.74 -60.96) (layer F.SilkS)
-      (effects (font (size 5.00126 5.00126) (thickness 0.50038)))
-    )
-    (fp_text value EuroBoard160mmX100mm_holes (at 85.09 -35.56) (layer F.SilkS)
-      (effects (font (size 5.00126 5.00126) (thickness 0.50038)))
-    )
-    (fp_line (start 1.00076 -99.9998) (end 0 -99.9998) (layer F.SilkS) (width 0.381))
-    (fp_line (start 0 -99.9998) (end 0 0) (layer Edge.Cuts) (width 0.381))
+  (module EuroBoard_viertel_Type-III_160mmX25mm (layer Vorderseite)
+    (at 73 42)
+    (descr "Outline, Eurocard 1/4, Type III,  160x25mm,")
+    (tags "Outline, Eurocard 1/4, Type III, 160x25mm,")
+    (fp_text reference Outl (at 75.5 -21) (layer F.SilkS)
+      (effects (font (size 2.99974 2.99974) (thickness 0.50038)))
+    )
+    (fp_text value EuroBoard_viertel_Type-III_160mmX25mm (at 87.5 -4.5) (layer F.SilkS)
+      (effects (font (size 3.00228 3.00228) (thickness 0.50038)))
+    )
     (fp_line (start 0 0) (end 159.99968 0) (layer Edge.Cuts) (width 0.381))
-    (fp_line (start 159.99968 0) (end 159.99968 -99.9998) (layer Edge.Cuts) (width 0.381))
-    (fp_line (start 159.99968 -99.9998) (end 1.00076 -99.9998) (layer Edge.Cuts) (width 0.381))
-    (pad 1 thru_hole circle (at 5.00126 -95.00108) (size 3.50012 3.50012) (drill 3.50012)
-      (layers *.Cu *.Mask F.SilkS)
-    )
-    (pad 2 thru_hole circle (at 155.00096 -95.00108) (size 3.50012 3.50012) (drill 3.50012)
-      (layers *.Cu *.Mask F.SilkS)
-    )
-    (pad 3 thru_hole circle (at 155.00096 -5.00126) (size 3.50012 3.50012) (drill 3.50012)
-      (layers *.Cu *.Mask F.SilkS)
-    )
-    (pad 4 thru_hole circle (at 5.00126 -5.00126) (size 3.50012 3.50012) (drill 3.50012)
-      (layers *.Cu *.Mask F.SilkS)
-    )
-  )
-  (module EuroBoard_achtel_Type-II_80mmX25mm_holes (layer Vorderseite)
-    (at 255.5 119 90)
-    (descr "Outline, Eurocard 1/8, Type II,  80x25mm, with holes 3,5mm,")
-    (tags "Outline, Eurocard 1/8, Type I, 80x25mm, with holes 3,5mm,")
-    (fp_text reference Outl (at 41.00068 -29.99994 90) (layer F.SilkS)
+    (fp_line (start 159.99968 0) (end 159.99968 -25.00122) (layer Edge.Cuts) (width 0.381))
+    (fp_line (start 159.99968 -25.00122) (end 0 -25.00122) (layer Edge.Cuts) (width 0.381))
+    (fp_line (start 0 -25.00122) (end 0 0) (layer Edge.Cuts) (width 0.381))
+  )
+  (module EuroBoard_viertel_Type-II_100mmX40mm (layer Vorderseite)
+    (at 58 125)
+    (descr "Outline, Eurocard 1/4, Type I, 100x40mm,")
+    (tags "Outline, Eurocard 1/4, Type II, 100x40mm,")
+    (fp_text reference Outl (at 52.5 -34.5) (layer F.SilkS)
       (effects (font (size 2.99974 2.99974) (thickness 0.50038)))
     )
-    (fp_text value EuroBoard_achtel_Type-II_80mmX25mm_holes (at 41.9989 5.99948 90) (layer F.SilkS)
+    (fp_text value EuroBoard_viertel_Type-II_100mmX40mm (at 48 3.5) (layer F.SilkS)
       (effects (font (size 3.00228 3.00228) (thickness 0.50038)))
     )
-    (fp_line (start 0 0) (end 79.99984 0) (layer Edge.Cuts) (width 0.381))
-    (fp_line (start 79.99984 0) (end 79.99984 -25.00122) (layer Edge.Cuts) (width 0.381))
-    (fp_line (start 79.99984 -25.00122) (end 0 -25.00122) (layer Edge.Cuts) (width 0.381))
+    (fp_line (start 0 0) (end 99.9998 0) (layer Edge.Cuts) (width 0.381))
+    (fp_line (start 99.9998 0) (end 99.9998 -39.99992) (layer Edge.Cuts) (width 0.381))
+    (fp_line (start 99.9998 -39.99992) (end 0 -39.99992) (layer Edge.Cuts) (width 0.381))
+    (fp_line (start 0 -39.99992) (end 0 0) (layer Edge.Cuts) (width 0.381))
+  )
+  (module EuroBoard_viertel_Type-III_160mmX25mm_holes (layer Vorderseite)
+    (at 73 75)
+    (descr "Outline, Eurocard 1/4, Type III,  160x25mm, with holes 3,5mm,")
+    (tags "Outline, Eurocard 1/4, Type III, 160x25mm, with holes 3,5mm,")
+    (fp_text reference Outl (at 70.5 -18.5) (layer F.SilkS)
+      (effects (font (size 2.99974 2.99974) (thickness 0.50038)))
+    )
+    (fp_text value EuroBoard_viertel_Type-III_160mmX25mm_holes (at 82 -10.5) (layer F.SilkS)
+      (effects (font (size 3.00228 3.00228) (thickness 0.50038)))
+    )
+    (fp_line (start 0 0) (end 159.99968 0) (layer Edge.Cuts) (width 0.381))
+    (fp_line (start 159.99968 0) (end 159.99968 -25.00122) (layer Edge.Cuts) (width 0.381))
+    (fp_line (start 159.99968 -25.00122) (end 0 -25.00122) (layer Edge.Cuts) (width 0.381))
     (fp_line (start 0 -25.00122) (end 0 0) (layer Edge.Cuts) (width 0.381))
-    (pad 1 thru_hole circle (at 5.00126 -5.00126 90) (size 3.50012 3.50012) (drill 3.50012)
-      (layers *.Cu *.Mask F.SilkS)
-    )
-    (pad 2 thru_hole circle (at 5.00126 -19.99996 90) (size 3.50012 3.50012) (drill 3.50012)
-      (layers *.Cu *.Mask F.SilkS)
-    )
-    (pad 3 thru_hole circle (at 75.00112 -19.99996 90) (size 3.50012 3.50012) (drill 3.50012)
-      (layers *.Cu *.Mask F.SilkS)
-    )
-    (pad 4 thru_hole circle (at 75.00112 -5.00126 90) (size 3.50012 3.50012) (drill 3.50012)
+    (pad "" np_thru_hole circle (at 5.00126 -5.00126) (size 3.50012 3.50012) (drill 3.50012)
+      (layers *.Cu *.Mask F.SilkS)
+    )
+    (pad "" np_thru_hole circle (at 5.00126 -19.99996) (size 3.50012 3.50012) (drill 3.50012)
+      (layers *.Cu *.Mask F.SilkS)
+    )
+    (pad "" np_thru_hole circle (at 79.99984 -19.99996) (size 3.50012 3.50012) (drill 3.50012)
+      (layers *.Cu *.Mask F.SilkS)
+    )
+    (pad "" np_thru_hole circle (at 155.00096 -19.99996) (size 3.50012 3.50012) (drill 3.50012)
+      (layers *.Cu *.Mask F.SilkS)
+    )
+    (pad "" np_thru_hole circle (at 155.00096 -5.00126) (size 3.50012 3.50012) (drill 3.50012)
+      (layers *.Cu *.Mask F.SilkS)
+    )
+    (pad "" np_thru_hole circle (at 79.99984 -5.00126) (size 3.50012 3.50012) (drill 3.50012)
+      (layers *.Cu *.Mask F.SilkS)
+    )
+  )
+  (module EuroBoard_viertel_Type-II_100mmX40mm_holes (layer Vorderseite)
+    (at 172.5 125)
+    (descr "Outline, Eurocard 1/4, Type I, 100x40mm, with holes 3,5mm,")
+    (tags "Outline, Eurocard 1/4, Type II, 100x40mm, with holes 3,5mm,")
+    (fp_text reference Outl (at 50.5 -35.5) (layer F.SilkS)
+      (effects (font (size 2.99974 2.99974) (thickness 0.50038)))
+    )
+    (fp_text value EuroBoard_viertel_Type-II_100mmX40mm_holes (at 51.00066 7.00024) (layer F.SilkS)
+      (effects (font (size 3.00228 3.00228) (thickness 0.50038)))
+    )
+    (fp_line (start 0 0) (end 99.9998 0) (layer Edge.Cuts) (width 0.381))
+    (fp_line (start 99.9998 0) (end 99.9998 -39.99992) (layer Edge.Cuts) (width 0.381))
+    (fp_line (start 99.9998 -39.99992) (end 0 -39.99992) (layer Edge.Cuts) (width 0.381))
+    (fp_line (start 0 -39.99992) (end 0 0) (layer Edge.Cuts) (width 0.381))
+    (pad "" np_thru_hole circle (at 5.00126 -5.00126) (size 3.50012 3.50012) (drill 3.50012)
+      (layers *.Cu *.Mask F.SilkS)
+    )
+    (pad "" np_thru_hole circle (at 5.00126 -35.0012) (size 3.50012 3.50012) (drill 3.50012)
+      (layers *.Cu *.Mask F.SilkS)
+    )
+    (pad "" np_thru_hole circle (at 95.00108 -35.0012) (size 3.50012 3.50012) (drill 3.50012)
+      (layers *.Cu *.Mask F.SilkS)
+    )
+    (pad "" np_thru_hole circle (at 95.00108 -5.00126) (size 3.50012 3.50012) (drill 3.50012)
       (layers *.Cu *.Mask F.SilkS)
     )
@@
     (effects (font (size 4.0005 4.0005) (thickness 0.59944)))
   )
-  (gr_text "Author: Bernd Wiebus / Uedem / Germany / 04 Jun 2013" (at 114.50012 172.24958) (layer F.SilkS)
+  (gr_text "Author: Bernd Wiebus / Uedem / Germany / 07 Jun 2013" (at 114.50012 172.24958) (layer F.SilkS)
     (effects (font (size 4.0005 4.0005) (thickness 0.59944)))
   )
-  (gr_text EuroBoardoutline_RevB.mod (at 114.00028 165.9989) (layer F.SilkS)
+  (gr_text EuroBoardoutline_RevC.mod (at 114.00028 165.9989) (layer F.SilkS)
     (effects (font (size 4.0005 4.0005) (thickness 0.59944)))
   )
