File: modules/OldSowjetAera_Transistor_RevA.kicad_pcb (KiCad board)
At the start: 2 copper layers, 5 parts

Commit message: Some new 3D models (7-Segment and BNC-socket) and some lost(???)  .mod files
Parts:
- added T: OldSowjetaera_Transistor_Type-II_BigPads_RevA, OldSowjetaera_Transistor_Type-II_BigPads_RevA, F.Cu at (232.0, 111.5)
- added T: OldSowjetaera_Transistor_Type-II_SmallPads_RevA, OldSowjetaera_Transistor_Type-II_SmallPads_RevA, F.Cu at (236.5, 85.0)
Other:
- board text added: "Author: Bernd Wiebus / Uedem / Germany / 12 July 2013"
- board text removed: "Author: Bernd Wiebus / Uedem / Germany / 28 May 2013"
Changed lines of the file:
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@@
     (links 0)
     (no_connects 0)
-    (area -16.90696 40.805099 274.02378 197.1694)
+    (area -16.90696 40.805099 276.799733 197.1694)
     (thickness 1.6002)
     (drawings 8)
     (tracks 0)
     (zones 0)
-    (modules 5)
+    (modules 7)
     (nets 1)
   )
@@
     )
   )
+  (module OldSowjetaera_Transistor_Type-II_BigPads_RevA (layer Vorderseite)
+    (at 232 111.5)
+    (fp_text reference T (at 0.1 -8.1) (layer F.SilkS)
+      (effects (font (size 1.524 1.524) (thickness 0.3048)))
+    )
+    (fp_text value OldSowjetaera_Transistor_Type-II_BigPads_RevA (at 0.1 7.6) (layer F.SilkS)
+      (effects (font (size 1.524 1.524) (thickness 0.3048)))
+    )
+    (fp_circle (center -4.8 0) (end -4.8 0.4) (layer F.SilkS) (width 0.381))
+    (fp_circle (center 0 0) (end 4 0) (layer F.SilkS) (width 0.381))
+    (fp_circle (center 0 0) (end 5.6 0) (layer F.SilkS) (width 0.381))
+    (pad 2 thru_hole oval (at 0 -2) (size 1.4 2.5) (drill 0.8)
+      (layers *.Cu *.Mask F.SilkS)
+    )
+    (pad 1 thru_hole oval (at -2 0 90) (size 1.4 2.5) (drill 0.8)
+      (layers *.Cu *.Mask F.SilkS)
+    )
+    (pad 3 thru_hole oval (at 2 0 90) (size 1.4 2.5) (drill 0.8)
+      (layers *.Cu *.Mask F.SilkS)
+    )
+    (model OldSowjetAera_Transistor_Type-II_Faktor03937_RevA.wrl
+      (at (xyz 0 0 0))
+      (scale (xyz 0.3937 0.3937 0.3937))
+      (rotate (xyz 0 0 0))
+    )
+  )
+  (module OldSowjetaera_Transistor_Type-II_SmallPads_RevA (layer Vorderseite)
+    (at 236.5 85)
+    (fp_text reference T (at 0 -7.1) (layer F.SilkS)
+      (effects (font (size 1.524 1.524) (thickness 0.3048)))
+    )
+    (fp_text value OldSowjetaera_Transistor_Type-II_SmallPads_RevA (at 0.1 7.6) (layer F.SilkS)
+      (effects (font (size 1.524 1.524) (thickness 0.3048)))
+    )
+    (fp_circle (center -4.8 0) (end -4.8 0.4) (layer F.SilkS) (width 0.381))
+    (fp_circle (center 0 0) (end 4 0) (layer F.SilkS) (width 0.381))
+    (fp_circle (center 0 0) (end 5.6 0) (layer F.SilkS) (width 0.381))
+    (pad 2 thru_hole circle (at 0 -2) (size 1.4 1.4) (drill 0.8)
+      (layers *.Cu *.Mask F.SilkS)
+    )
+    (pad 1 thru_hole circle (at -2 0) (size 1.4 1.4) (drill 0.8)
+      (layers *.Cu *.Mask F.SilkS)
+    )
+    (pad 3 thru_hole circle (at 2 0) (size 1.4 1.4) (drill 0.8)
+      (layers *.Cu *.Mask F.SilkS)
+    )
+    (model OldSowjetAera_Transistor_Type-II_Faktor03937_RevA.wrl
+      (at (xyz 0 0 0))
+      (scale (xyz 0.3937 0.3937 0.3937))
+      (rotate (xyz 0 0 0))
+    )
+  )
   (gr_text "There is no official pin numbering for this type of footprint!\nSo i had to choose a numbering at random.\nSo it starts with one at the pin nearest to the black dot.\nPin two is the middle pin, and pin thre the last.\n\nBe careful and check your allocation!" (at 218 54) (layer Vorderseite)
     (effects (font (size 2.032 1.524) (thickness 0.3048) italic))
@@
     (effects (font (size 4.0005 4.0005) (thickness 0.59944)))
   )
-  (gr_text "Author: Bernd Wiebus / Uedem / Germany / 28 May 2013  " (at 114.50012 172.24958) (layer F.SilkS)
+  (gr_text "Author: Bernd Wiebus / Uedem / Germany / 12 July 2013  " (at 114.50012 172.24958) (layer F.SilkS)
     (effects (font (size 4.0005 4.0005) (thickness 0.59944)))
   )
