File: modules/NF-Transformer_ETAL_RevA_28Aug2012.kicad_pcb (KiCad board)
At the start: 2 copper layers, 17 parts

Commit message: Some minor impovements to 3D models.
Parts:
- moved TR 5.64 mm to (188.8, 29.5)
