File: modules/LEM_HallEffectTransducers_RevA_13Oct2012.kicad_pcb (KiCad board)
At the start: 2 copper layers, 9 parts

Commit message: Footprind and 3d modell of LEM HTFS-series hall effect current transducers added.
Parts:
- added U: HTFS-Series_LEM-HallEffektCurrentTransducer_RevA_16Oct2013, HTFS-Series_LEM-HallEffektCurrentTransducer_RevA_16Oct2013, F.Cu at (235.5, 60.2)
- moved U 147.8 mm to (62.0, 135.0)
- moved U 31.4 mm to (172.0, 49.2)
- moved U 17.4 mm to (63.8, 107.5)
- moved U 16.9 mm to (62.0, 77.2)
- moved U 15.9 mm to (62.8, 44.8)
- moved U 11.9 mm to (173.8, 105.8)
