File: modules/Buzzer_Beeper_RevA_25Oct2010.kicad_pcb (KiCad board)
At the start: 2 copper layers, 7 parts

Commit message: Updates for pretty folders.
Parts:
- added Sym: Symbol_CreativeCommonsPublicDomain_SilkScreenTop_Small, Symbols:Symbol_CreativeCommonsPublicDomain_SilkScreenTop_Small, F.Cu at (71.0, 186.5)
Other:
- board text added: "Buzzer_Beeper_RevA_25Oct2010.pretty (was Buzzer_Beeper_RevA_25Oct2010.mod)"
- board text added: "KiCAD Footprints of some buzzers and beepers from the folder"
- board text removed: "Buzzer_Beeper_RevA_25Oct2010.mod"
- board text removed: "KiCAD Footprints of some buzzers and beepers from the file"
