File: modules/Choke_Radial_ThroughHole_CD_Bobin_RevA.kicad_pcb (KiCad board)
At the start: 2 copper layers, 7 parts

Commit message: Updates for pretty folders.
Other:
- board text added: "Choke_Radial_ThroughHole_CD_Bobin_RevA.pretty (was Choke_Radial_ThroughHole_CD_Bobin_RevA.mod)"
- board text added: "KiCAD Footprints of some radial chokes (Manufactured by C&D) from the folder"
- board text removed: "Choke_Radial_ThroughHole_CD_Bobin_RevA.mod"
- board text removed: "KiCAD Footprints of some radial chokes (Manufactured by C&D) from the file"
Changed lines of the file:
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@@
-(kicad_pcb (version 3) (host pcbnew "(2013-03-30 BZR 4007)-stable")
+(kicad_pcb (version 3) (host pcbnew "(2014-02-28 BZR 4727)-product")
   (general
     (links 0)
     (no_connects 0)
-    (area -4.90696 -58.199132 267.98147 197.6694)
+    (area 4.382182 -58.199132 267.98147 197.9742)
     (thickness 1.6002)
     (drawings 8)
@@
       (usegerberextensions true)
       (excludeedgelayer true)
-      (linewidth 60)
+      (linewidth 0.150000)
       (plotframeref false)
       (viasonmask false)
@@
     (path Gauge_100mm_Type2_SilkScreenTop_RevA_Date22Jun2010)
     (fp_text reference MSC (at 4.0005 8.99922) (layer F.SilkS) hide
-      (effects (font (size 1.524 1.524) (thickness 0.3048)))
+      (effects (font (thickness 0.3048)))
     )
     (fp_text value Gauge_100mm_Type2_SilkScreenTop_RevA_Date22Jun2010 (at 45.9994 8.99922) (layer F.SilkS) hide
-      (effects (font (size 1.524 1.524) (thickness 0.3048)))
+      (effects (font (thickness 0.3048)))
     )
     (fp_text user mm (at 9.99998 5.00126) (layer F.SilkS)
-      (effects (font (size 1.524 1.524) (thickness 0.3048)))
+      (effects (font (thickness 0.3048)))
     )
     (fp_text user mm (at -4.0005 -8.99922) (layer F.SilkS)
-      (effects (font (size 1.524 1.524) (thickness 0.3048)))
+      (effects (font (thickness 0.3048)))
     )
     (fp_text user mm (at -5.00126 -98.5012) (layer F.SilkS)
-      (effects (font (size 1.524 1.524) (thickness 0.3048)))
+      (effects (font (thickness 0.3048)))
     )
     (fp_text user 10 (at 10.00506 3.0988) (layer F.SilkS)
@@
     (tags "Choke, Radial, Bobin Type, Diameter, 27mm, 2.8mm Drill, C&D, No.1410311, 22uH, 11A,")
     (fp_text reference L (at 0.254 -15.367) (layer F.SilkS)
-      (effects (font (size 1.524 1.524) (thickness 0.3048)))
+      (effects (font (thickness 0.3048)))
     )
     (fp_text value Choke_22uH/11A_C&D_Bobin_Type_No1410311 (at 1.905 14.986) (layer F.SilkS)
-      (effects (font (size 1.524 1.524) (thickness 0.3048)))
+      (effects (font (thickness 0.3048)))
     )
     (fp_line (start -11.684 -3.048) (end -11.43 -3.937) (layer F.SilkS) (width 0.381))
@@
     (fp_line (start 14.859 -1.27) (end 15.113 -0.508) (layer F.SilkS) (width 0.381))
     (fp_line (start 15.113 -0.508) (end 15.113 0) (layer F.SilkS) (width 0.381))
-    (pad 1 thru_hole circle (at 12.065 0) (size 5.00126 5.00126) (drill 2.79908)
-      (layers *.Cu *.Mask F.SilkS)
-    )
-    (pad 2 thru_hole circle (at -12.065 0) (size 5.00126 5.00126) (drill 2.79908)
-      (layers *.Cu *.Mask F.SilkS)
-    )
+    (pad 1 thru_hole circle (at 12.065 0) (size 5.00126 5.00126) (drill 2.79908) (layers *.Cu *.Mask F.SilkS))
+    (pad 2 thru_hole circle (at -12.065 0) (size 5.00126 5.00126) (drill 2.79908) (layers *.Cu *.Mask F.SilkS))
   )
   (module Choke_Radial_27mm_2,8mm-Drills_CD_Bobin_Type_No1410312 (layer Vorderseite)
@@
     (tags "Choke, Radial, Bobin Type, Diameter, 27mm, 2.8mm Drill, C&D, No.1410312, 15uH, 12A,")
     (fp_text reference L (at 0.254 -15.367) (layer F.SilkS)
-      (effects (font (size 1.524 1.524) (thickness 0.3048)))
+      (effects (font (thickness 0.3048)))
     )
     (fp_text value Choke_15uH/12A_DM27mm_C&D_Bobin_Type_No1410312 (at 1.905 14.986) (layer F.SilkS)
-      (effects (font (size 1.524 1.524) (thickness 0.3048)))
+      (effects (font (thickness 0.3048)))
     )
     (fp_line (start -11.684 -3.048) (end -11.43 -3.937) (layer F.SilkS) (width 0.381))
@@
     (fp_line (start 14.859 -1.27) (end 15.113 -0.508) (layer F.SilkS) (width 0.381))
     (fp_line (start 15.113 -0.508) (end 15.113 0) (layer F.SilkS) (width 0.381))
-    (pad 1 thru_hole circle (at 12.065 0) (size 5.00126 5.00126) (drill 2.79908)
-      (layers *.Cu *.Mask F.SilkS)
-    )
-    (pad 2 thru_hole circle (at -12.065 0) (size 5.00126 5.00126) (drill 2.79908)
-      (layers *.Cu *.Mask F.SilkS)
-    )
+    (pad 1 thru_hole circle (at 12.065 0) (size 5.00126 5.00126) (drill 2.79908) (layers *.Cu *.Mask F.SilkS))
+    (pad 2 thru_hole circle (at -12.065 0) (size 5.00126 5.00126) (drill 2.79908) (layers *.Cu *.Mask F.SilkS))
   )
   (module Choke_Radial_31mm_1.5mm-Drills_CD_Bobin_Type_No1410514 (layer Vorderseite)
@@
     (tags "Choke, Radial, Bobin Type, Diameter 31mm, C&D, No.1410514, Drossel, Spule, Durchmesser, 1.5mm Drill, Bohrung, 2.2mH, 1.4A,")
     (fp_text reference L (at 0 -2.413) (layer F.SilkS)
-      (effects (font (size 1.524 1.524) (thickness 0.3048)))
+      (effects (font (thickness 0.3048)))
     )
     (fp_text value Choke_2.2mH/1.4A_C&D_No1410514_1.5mm_Drills (at -0.635 16.51) (layer F.SilkS)
-      (effects (font (size 1.524 1.524) (thickness 0.3048)))
+      (effects (font (thickness 0.3048)))
     )
     (fp_line (start -13.462 -2.921) (end -13.208 -3.937) (layer F.SilkS) (width 0.381))
@@
     (fp_line (start 12.954 6.731) (end 11.557 8.89) (layer F.SilkS) (width 0.381))
     (fp_line (start 11.557 8.89) (end 9.525 11.049) (layer F.SilkS) (width 0.381))
-    (pad 1 thru_hole circle (at 14.605 0) (size 5.00126 5.00126) (drill 1.50114)
-      (layers *.Cu *.Mask F.SilkS)
-    )
-    (pad 2 thru_hole circle (at -14.605 0) (size 5.00126 5.00126) (drill 1.50114)
-      (layers *.Cu *.Mask F.SilkS)
-    )
+    (pad 1 thru_hole circle (at 14.605 0) (size 5.00126 5.00126) (drill 1.50114) (layers *.Cu *.Mask F.SilkS))
+    (pad 2 thru_hole circle (at -14.605 0) (size 5.00126 5.00126) (drill 1.50114) (layers *.Cu *.Mask F.SilkS))
   )
   (module Choke_Radial_31mm_2.4mm-Drills_CD_Bobin_Type_No1422455 (layer Vorderseite)
@@
     (tags "Choke, Radial, Bobin Type, Diameter 31mm, C&D, No.1422455, Drossel, Spule, Durchmesser, 2.4mm Drill, Bohrung, 220uH, 5.5A,")
     (fp_text reference L (at 0 -2.413) (layer F.SilkS)
-      (effects (font (size 1.524 1.524) (thickness 0.3048)))
+      (effects (font (thickness 0.3048)))
     )
     (fp_text value Choke_220uH/5.5A_C&D_No1422455_2.4mm_Drills (at -0.635 16.51) (layer F.SilkS)
-      (effects (font (size 1.524 1.524) (thickness 0.3048)))
+      (effects (font (thickness 0.3048)))
     )
     (fp_line (start -13.462 -2.921) (end -13.208 -3.937) (layer F.SilkS) (width 0.381))
@@
     (fp_line (start 12.954 6.731) (end 11.557 8.89) (layer F.SilkS) (width 0.381))
     (fp_line (start 11.557 8.89) (end 9.525 11.049) (layer F.SilkS) (width 0.381))
-    (pad 1 thru_hole circle (at 14.605 0) (size 5.00126 5.00126) (drill 2.4003)
-      (layers *.Cu *.Mask F.SilkS)
-    )
-    (pad 2 thru_hole circle (at -14.605 0) (size 5.00126 5.00126) (drill 2.4003)
-      (layers *.Cu *.Mask F.SilkS)
-    )
+    (pad 1 thru_hole circle (at 14.605 0) (size 5.00126 5.00126) (drill 2.4003) (layers *.Cu *.Mask F.SilkS))
+    (pad 2 thru_hole circle (at -14.605 0) (size 5.00126 5.00126) (drill 2.4003) (layers *.Cu *.Mask F.SilkS))
   )
   (module Symbol_CC-PublicDomain_SilkScreenTop_Big (layer Vorderseite)
@@
     (path Symbol_CC-Noncommercial_CopperTop_Big)
     (fp_text reference Sym (at 0.59944 -7.29996) (layer F.SilkS) hide
-      (effects (font (size 1.524 1.524) (thickness 0.3048)))
+      (effects (font (thickness 0.3048)))
     )
     (fp_text value Symbol_CC-PublicDomain_SilkScreenTop_Big (at 0.59944 8.001) (layer F.SilkS) hide
-      (effects (font (size 1.524 1.524) (thickness 0.3048)))
+      (effects (font (thickness 0.3048)))
     )
     (fp_circle (center 0 0) (end 5.8 -0.05) (layer F.SilkS) (width 0.381))
@@
     (path Symbol_CreativeCommons_CopperTop_Type2_Big)
     (fp_text reference Sym (at 0.59944 -7.29996) (layer F.SilkS) hide
-      (effects (font (size 1.524 1.524) (thickness 0.3048)))
+      (effects (font (thickness 0.3048)))
     )
     (fp_text value Symbol_CreativeCommons_Typ2_SilkScreenTop_Big (at 0.59944 8.001) (layer F.SilkS) hide
-      (effects (font (size 1.524 1.524) (thickness 0.3048)))
+      (effects (font (thickness 0.3048)))
     )
     (fp_line (start -0.70104 2.70002) (end -0.29972 2.60096) (layer F.SilkS) (width 0.381))
@@
     (effects (font (size 4.0005 4.0005) (thickness 0.59944)))
   )
-  (gr_text "Author: Bernd Wiebus / Uedem / Germany / 20th Oct 2010" (at 125.50012 172.74958) (layer F.SilkS)
+  (gr_text "Author: Bernd Wiebus / Uedem / Germany / 20th Oct 2010" (at 94.5 168.5) (layer F.SilkS)
+    (effects (font (size 4.0005 3.5) (thickness 0.59944)))
+  )
+  (gr_text "Choke_Radial_ThroughHole_CD_Bobin_RevA.pretty (was Choke_Radial_ThroughHole_CD_Bobin_RevA.mod)" (at 149 161) (layer F.SilkS)
+    (effects (font (size 4.0005 3.3) (thickness 0.59944)))
+  )
+  (gr_text "KiCAD Footprints of some radial chokes (Manufactured by C&D) from the folder" (at 146.5 154) (layer F.SilkS)
     (effects (font (size 4.0005 4.0005) (thickness 0.59944)))
   )
-  (gr_text Choke_Radial_ThroughHole_CD_Bobin_RevA.mod (at 125.00028 166.4989) (layer F.SilkS)
-    (effects (font (size 4.0005 4.0005) (thickness 0.59944)))
-  )
-  (gr_text "KiCAD Footprints of some radial chokes (Manufactured by C&D) from the file " (at 147 157) (layer F.SilkS)
-    (effects (font (size 4.0005 4.0005) (thickness 0.59944)))
-  )
