File: template/Arduino_As_Uno_R3/Arduino_As_Uno.kicad_pcb (KiCad board)
At the start: 2 copper layers, 68.6 x 53.3 mm, 8 parts, among them P1 Power, P2 Analog, P3 Digital, P4 Digital, P5 CONN_1, P6 CONN_1, P7 CONN_1, P8 CONN_1

Commit message: corrections
Connections:
- net +3.3V renamed +3V3
- net /11(**/MISO) renamed /11(**/MOSI)
- net /12(MOSI) renamed /12(MISO)
- net /NC renamed Net-(P1-Pad1)
Other:
- board text added: "1"
Changed lines of the file:
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@@
     (links 4)
     (no_connects 4)
-    (area 110.922999 72.949999 179.653001 126.440001)
+    (area 104.572999 71.392 180.241572 127.594)
     (thickness 1.6)
-    (drawings 26)
+    (drawings 27)
     (tracks 0)
     (zones 0)
@@
   )
   (net 0 "")
-  (net 1 /NC)
-  (net 2 /IOREF)
-  (net 3 /Reset)
-  (net 4 +3.3V)
-  (net 5 +5V)
-  (net 6 GND)
-  (net 7 /Vin)
-  (net 8 /A0)
-  (net 9 /A1)
-  (net 10 /A2)
-  (net 11 /A3)
-  (net 12 /AREF)
-  (net 13 "/A4(SDA)")
-  (net 14 "/A5(SCL)")
-  (net 15 "/9(**)")
-  (net 16 /8)
-  (net 17 /7)
-  (net 18 "/6(**)")
-  (net 19 "/5(**)")
-  (net 20 /4)
-  (net 21 "/3(**)")
-  (net 22 /2)
-  (net 23 "/1(Tx)")
-  (net 24 "/0(Rx)")
-  (net 25 "Net-(P5-Pad1)")
-  (net 26 "Net-(P6-Pad1)")
-  (net 27 "Net-(P7-Pad1)")
-  (net 28 "Net-(P8-Pad1)")
-  (net 29 "/13(SCK)")
-  (net 30 "/12(MOSI)")
-  (net 31 "/11(**/MISO)")
-  (net 32 "/10(**/SS)")
+  (net 1 /IOREF)
+  (net 2 /Reset)
+  (net 3 +5V)
+  (net 4 GND)
+  (net 5 /Vin)
+  (net 6 /A0)
+  (net 7 /A1)
+  (net 8 /A2)
+  (net 9 /A3)
+  (net 10 /AREF)
+  (net 11 "/A4(SDA)")
+  (net 12 "/A5(SCL)")
+  (net 13 "/9(**)")
+  (net 14 /8)
+  (net 15 /7)
+  (net 16 "/6(**)")
+  (net 17 "/5(**)")
+  (net 18 /4)
+  (net 19 "/3(**)")
+  (net 20 /2)
+  (net 21 "/1(Tx)")
+  (net 22 "/0(Rx)")
+  (net 23 "Net-(P5-Pad1)")
+  (net 24 "Net-(P6-Pad1)")
+  (net 25 "Net-(P7-Pad1)")
+  (net 26 "Net-(P8-Pad1)")
+  (net 27 "/13(SCK)")
+  (net 28 "/10(**/SS)")
+  (net 29 "Net-(P1-Pad1)")
+  (net 30 +3V3)
+  (net 31 "/12(MISO)")
+  (net 32 "/11(**/MOSI)")
   (net_class Default "This is the default net class."
     (clearance 0.2)
@@
     (uvia_dia 0.3)
     (uvia_drill 0.1)
-    (add_net +3.3V)
+    (add_net +3V3)
     (add_net +5V)
     (add_net "/0(Rx)")
     (add_net "/1(Tx)")
     (add_net "/10(**/SS)")
-    (add_net "/11(**/MISO)")
-    (add_net "/12(MOSI)")
+    (add_net "/11(**/MOSI)")
+    (add_net "/12(MISO)")
     (add_net "/13(SCK)")
     (add_net /2)
@@
     (add_net /AREF)
     (add_net /IOREF)
-    (add_net /NC)
     (add_net /Reset)
     (add_net /Vin)
     (add_net GND)
+    (add_net "Net-(P1-Pad1)")
     (add_net "Net-(P5-Pad1)")
     (add_net "Net-(P6-Pad1)")
@@
     (fp_line (start -1.55 -1.55) (end -1.55 1.55) (layer F.SilkS) (width 0.15))
     (pad 1 thru_hole oval (at 0 0) (size 1.7272 2.032) (drill 1.016) (layers *.Cu *.Mask F.SilkS)
-      (net 1 /NC))
+      (net 29 "Net-(P1-Pad1)"))
     (pad 2 thru_hole oval (at 2.54 0) (size 1.7272 2.032) (drill 1.016) (layers *.Cu *.Mask F.SilkS)
-      (net 2 /IOREF))
+      (net 1 /IOREF))
     (pad 3 thru_hole oval (at 5.08 0) (size 1.7272 2.032) (drill 1.016) (layers *.Cu *.Mask F.SilkS)
-      (net 3 /Reset))
+      (net 2 /Reset))
     (pad 4 thru_hole oval (at 7.62 0) (size 1.7272 2.032) (drill 1.016) (layers *.Cu *.Mask F.SilkS)
-      (net 4 +3.3V))
+      (net 30 +3V3))
     (pad 5 thru_hole oval (at 10.16 0) (size 1.7272 2.032) (drill 1.016) (layers *.Cu *.Mask F.SilkS)
-      (net 5 +5V))
+      (net 3 +5V))
     (pad 6 thru_hole oval (at 12.7 0) (size 1.7272 2.032) (drill 1.016) (layers *.Cu *.Mask F.SilkS)
-      (net 6 GND))
+      (net 4 GND))
     (pad 7 thru_hole oval (at 15.24 0) (size 1.7272 2.032) (drill 1.016) (layers *.Cu *.Mask F.SilkS)
-      (net 6 GND))
+      (net 4 GND))
     (pad 8 thru_hole oval (at 17.78 0) (size 1.7272 2.032) (drill 1.016) (layers *.Cu *.Mask F.SilkS)
-      (net 7 /Vin))
+      (net 5 /Vin))
     (model ${KIPRJMOD}/Socket_Arduino_Uno.3dshapes/Socket_header_Arduino_1x08.wrl
       (at (xyz 0.35 0 0))
@@
     (fp_line (start -1.55 -1.55) (end -1.55 1.55) (layer F.SilkS) (width 0.15))
     (pad 1 thru_hole oval (at 0 0) (size 1.7272 2.032) (drill 1.016) (layers *.Cu *.Mask F.SilkS)
-      (net 8 /A0))
+      (net 6 /A0))
     (pad 2 thru_hole oval (at 2.54 0) (size 1.7272 2.032) (drill 1.016) (layers *.Cu *.Mask F.SilkS)
-      (net 9 /A1))
+      (net 7 /A1))
     (pad 3 thru_hole oval (at 5.08 0) (size 1.7272 2.032) (drill 1.016) (layers *.Cu *.Mask F.SilkS)
-      (net 10 /A2))
+      (net 8 /A2))
     (pad 4 thru_hole oval (at 7.62 0) (size 1.7272 2.032) (drill 1.016) (layers *.Cu *.Mask F.SilkS)
-      (net 11 /A3))
+      (net 9 /A3))
     (pad 5 thru_hole oval (at 10.16 0) (size 1.7272 2.032) (drill 1.016) (layers *.Cu *.Mask F.SilkS)
-      (net 13 "/A4(SDA)"))
+      (net 11 "/A4(SDA)"))
     (pad 6 thru_hole oval (at 12.7 0) (size 1.7272 2.032) (drill 1.016) (layers *.Cu *.Mask F.SilkS)
-      (net 14 "/A5(SCL)"))
+      (net 12 "/A5(SCL)"))
     (model ${KIPRJMOD}/Socket_Arduino_Uno.3dshapes/Socket_header_Arduino_1x06.wrl
       (at (xyz 0.25 0 0))
@@
     (fp_line (start -1.55 -1.55) (end -1.55 1.55) (layer F.SilkS) (width 0.15))
     (pad 1 thru_hole oval (at 0 0) (size 1.7272 2.032) (drill 1.016) (layers *.Cu *.Mask F.SilkS)
-      (net 14 "/A5(SCL)"))
+      (net 12 "/A5(SCL)"))
     (pad 2 thru_hole oval (at 2.54 0) (size 1.7272 2.032) (drill 1.016) (layers *.Cu *.Mask F.SilkS)
-      (net 13 "/A4(SDA)"))
+      (net 11 "/A4(SDA)"))
     (pad 3 thru_hole oval (at 5.08 0) (size 1.7272 2.032) (drill 1.016) (layers *.Cu *.Mask F.SilkS)
-      (net 12 /AREF))
+      (net 10 /AREF))
     (pad 4 thru_hole oval (at 7.62 0) (size 1.7272 2.032) (drill 1.016) (layers *.Cu *.Mask F.SilkS)
-      (net 6 GND))
+      (net 4 GND))
     (pad 5 thru_hole oval (at 10.16 0) (size 1.7272 2.032) (drill 1.016) (layers *.Cu *.Mask F.SilkS)
-      (net 29 "/13(SCK)"))
+      (net 27 "/13(SCK)"))
     (pad 6 thru_hole oval (at 12.7 0) (size 1.7272 2.032) (drill 1.016) (layers *.Cu *.Mask F.SilkS)
-      (net 30 "/12(MOSI)"))
+      (net 31 "/12(MISO)"))
     (pad 7 thru_hole oval (at 15.24 0) (size 1.7272 2.032) (drill 1.016) (layers *.Cu *.Mask F.SilkS)
-      (net 31 "/11(**/MISO)"))
+      (net 32 "/11(**/MOSI)"))
     (pad 8 thru_hole oval (at 17.78 0) (size 1.7272 2.032) (drill 1.016) (layers *.Cu *.Mask F.SilkS)
-      (net 32 "/10(**/SS)"))
+      (net 28 "/10(**/SS)"))
     (pad 9 thru_hole oval (at 20.32 0) (size 1.7272 2.032) (drill 1.016) (layers *.Cu *.Mask F.SilkS)
-      (net 15 "/9(**)"))
+      (net 13 "/9(**)"))
     (pad 10 thru_hole oval (at 22.86 0) (size 1.7272 2.032) (drill 1.016) (layers *.Cu *.Mask F.SilkS)
-      (net 16 /8))
+      (net 14 /8))
     (model ${KIPRJMOD}/Socket_Arduino_Uno.3dshapes/Socket_header_Arduino_1x10.wrl
       (at (xyz 0.45 0 0))
@@
     (fp_line (start -1.55 -1.55) (end -1.55 1.55) (layer F.SilkS) (width 0.15))
     (pad 1 thru_hole oval (at 0 0) (size 1.7272 2.032) (drill 1.016) (layers *.Cu *.Mask F.SilkS)
-      (net 17 /7))
+      (net 15 /7))
     (pad 2 thru_hole oval (at 2.54 0) (size 1.7272 2.032) (drill 1.016) (layers *.Cu *.Mask F.SilkS)
-      (net 18 "/6(**)"))
+      (net 16 "/6(**)"))
     (pad 3 thru_hole oval (at 5.08 0) (size 1.7272 2.032) (drill 1.016) (layers *.Cu *.Mask F.SilkS)
-      (net 19 "/5(**)"))
+      (net 17 "/5(**)"))
     (pad 4 thru_hole oval (at 7.62 0) (size 1.7272 2.032) (drill 1.016) (layers *.Cu *.Mask F.SilkS)
-      (net 20 /4))
+      (net 18 /4))
     (pad 5 thru_hole oval (at 10.16 0) (size 1.7272 2.032) (drill 1.016) (layers *.Cu *.Mask F.SilkS)
-      (net 21 "/3(**)"))
+      (net 19 "/3(**)"))
     (pad 6 thru_hole oval (at 12.7 0) (size 1.7272 2.032) (drill 1.016) (layers *.Cu *.Mask F.SilkS)
-      (net 22 /2))
+      (net 20 /2))
     (pad 7 thru_hole oval (at 15.24 0) (size 1.7272 2.032) (drill 1.016) (layers *.Cu *.Mask F.SilkS)
-      (net 23 "/1(Tx)"))
+      (net 21 "/1(Tx)"))
     (pad 8 thru_hole oval (at 17.78 0) (size 1.7272 2.032) (drill 1.016) (layers *.Cu *.Mask F.SilkS)
-      (net 24 "/0(Rx)"))
+      (net 22 "/0(Rx)"))
     (model ${KIPRJMOD}/Socket_Arduino_Uno.3dshapes/Socket_header_Arduino_1x08.wrl
       (at (xyz 0.35 0 0))
@@
     (fp_circle (center 0 0) (end 0 -2.286) (layer F.SilkS) (width 0.15))
     (pad 1 thru_hole circle (at 0 0) (size 4.064 4.064) (drill 3.048) (layers *.Cu *.Mask F.SilkS)
-      (net 25 "Net-(P5-Pad1)"))
+      (net 23 "Net-(P5-Pad1)"))
   )
   (module Connect:1pin (layer F.Cu)
@@
     (fp_circle (center 0 0) (end 0 -2.286) (layer F.SilkS) (width 0.15))
     (pad 1 thru_hole circle (at 0 0) (size 4.064 4.064) (drill 3.048) (layers *.Cu *.Mask F.SilkS)
-      (net 26 "Net-(P6-Pad1)"))
+      (net 24 "Net-(P6-Pad1)"))
   )
   (module Connect:1pin (layer F.Cu)
@@
     (fp_circle (center 0 0) (end 0 -2.286) (layer F.SilkS) (width 0.15))
     (pad 1 thru_hole circle (at 0 0) (size 4.064 4.064) (drill 3.048) (layers *.Cu *.Mask F.SilkS)
-      (net 27 "Net-(P7-Pad1)"))
+      (net 25 "Net-(P7-Pad1)"))
   )
   (module Connect:1pin (layer F.Cu)
@@
     (fp_circle (center 0 0) (end 0 -2.286) (layer F.SilkS) (width 0.15))
     (pad 1 thru_hole circle (at 0 0) (size 4.064 4.064) (drill 3.048) (layers *.Cu *.Mask F.SilkS)
-      (net 28 "Net-(P8-Pad1)"))
+      (net 26 "Net-(P8-Pad1)"))
+  )
+  (gr_text 1 (at 139.065 126.619) (layer Dwgs.User)
+    (effects (font (size 1.5 1.5) (thickness 0.3)))
   )
   (gr_circle (center 117.348 76.962) (end 118.618 76.962) (layer Dwgs.User) (width 0.15))
