File: template/Arduino_Mega_R3/Arduino_Mega.kicad_pcb (KiCad board)
At the start: 2 copper layers, 101.6 x 53.3 mm, 13 parts, among them P1 Digital, P2 Power, P3 Analog, P4 Analog, P5 PWM, P6 PWM, P7 Communication

Commit message: correction holes
Parts:
- removed REF** (x6): 1pin, Connect:1pin
- added P10: CONN_1, Connect:1pin, F.Cu at (199.9, 119.1)
- added P11: CONN_1, Connect:1pin, F.Cu at (118.6, 70.9)
- added P12: CONN_1, Connect:1pin, F.Cu at (169.4, 86.1)
- added P13: CONN_1, Connect:1pin, F.Cu at (193.5, 70.9)
- added P8: CONN_1, Connect:1pin, F.Cu at (117.3, 119.1)
- added P9: CONN_1, Connect:1pin, F.Cu at (169.4, 114.0)
Changed lines of the file:
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@@
     (links 6)
     (no_connects 6)
-    (area 96.952999 66.693 205.053001 122.895)
+    (area 103.302999 68.250999 205.053001 121.741001)
     (thickness 1.6)
     (drawings 26)
@@
     (zones 0)
     (modules 13)
-    (nets 81)
+    (nets 87)
   )
   (page A4)
@@
   (net 79 "/20(SDA)")
   (net 80 "/21(SCL)")
+  (net 81 "Net-(P8-Pad1)")
+  (net 82 "Net-(P9-Pad1)")
+  (net 83 "Net-(P10-Pad1)")
+  (net 84 "Net-(P11-Pad1)")
+  (net 85 "Net-(P12-Pad1)")
+  (net 86 "Net-(P13-Pad1)")
   (net_class Default "This is the default net class."
     (clearance 0.2)
@@
     (add_net /Vin)
     (add_net GND)
+    (add_net "Net-(P10-Pad1)")
+    (add_net "Net-(P11-Pad1)")
+    (add_net "Net-(P12-Pad1)")
+    (add_net "Net-(P13-Pad1)")
+    (add_net "Net-(P8-Pad1)")
+    (add_net "Net-(P9-Pad1)")
   )
   (module Socket_Arduino_Mega:Socket_Strip_Arduino_2x18 (layer F.Cu)
@@
   )
   (module Connect:1pin (layer F.Cu)
+    (at 117.348 119.126)
+    (descr "module 1 pin (ou trou mecanique de percage)")
+    (tags DEV)
+    (fp_text reference P8 (at 0 -3.048) (layer F.SilkS) hide
+      (effects (font (size 1 1) (thickness 0.15)))
+    )
+    (fp_text value CONN_1 (at 0 2.794) (layer F.Fab) hide
+      (effects (font (size 1 1) (thickness 0.15)))
+    )
+    (fp_circle (center 0 0) (end 0 -2.286) (layer F.SilkS) (width 0.15))
+    (pad "" thru_hole circle (at 0 0) (size 4.064 4.064) (drill 3.048) (layers *.Cu *.Mask F.SilkS)
+      (net 81 "Net-(P8-Pad1)"))
+  )
+  (module Connect:1pin (layer F.Cu)
+    (at 169.418 114.046)
+    (descr "module 1 pin (ou trou mecanique de percage)")
+    (tags DEV)
+    (fp_text reference P9 (at 0 -3.048) (layer F.SilkS) hide
+      (effects (font (size 1 1) (thickness 0.15)))
+    )
+    (fp_text value CONN_1 (at 0 2.794) (layer F.Fab) hide
+      (effects (font (size 1 1) (thickness 0.15)))
+    )
+    (fp_circle (center 0 0) (end 0 -2.286) (layer F.SilkS) (width 0.15))
+    (pad "" thru_hole circle (at 0 0) (size 4.064 4.064) (drill 3.048) (layers *.Cu *.Mask F.SilkS)
+      (net 82 "Net-(P9-Pad1)"))
+  )
+  (module Connect:1pin (layer F.Cu)
+    (at 199.898 119.126)
+    (descr "module 1 pin (ou trou mecanique de percage)")
+    (tags DEV)
+    (fp_text reference P10 (at 0 -3.048) (layer F.SilkS) hide
+      (effects (font (size 1 1) (thickness 0.15)))
+    )
+    (fp_text value CONN_1 (at 0 2.794) (layer F.Fab) hide
+      (effects (font (size 1 1) (thickness 0.15)))
+    )
+    (fp_circle (center 0 0) (end 0 -2.286) (layer F.SilkS) (width 0.15))
+    (pad "" thru_hole circle (at 0 0) (size 4.064 4.064) (drill 3.048) (layers *.Cu *.Mask F.SilkS)
+      (net 83 "Net-(P10-Pad1)"))
+  )
+  (module Connect:1pin (layer F.Cu)
     (at 118.618 70.866)
     (descr "module 1 pin (ou trou mecanique de percage)")
     (tags DEV)
-    (fp_text reference REF** (at 0 -3.048) (layer F.SilkS) hide
-      (effects (font (size 1 1) (thickness 0.15)))
-    )
-    (fp_text value 1pin (at 0 2.794) (layer F.Fab) hide
+    (fp_text reference P11 (at 0 -3.048) (layer F.SilkS) hide
+      (effects (font (size 1 1) (thickness 0.15)))
+    )
+    (fp_text value CONN_1 (at 0 2.794) (layer F.Fab) hide
       (effects (font (size 1 1) (thickness 0.15)))
     )
     (fp_circle (center 0 0) (end 0 -2.286) (layer F.SilkS) (width 0.15))
-    (pad "" thru_hole circle (at 0 0) (size 4.064 4.064) (drill 3.048) (layers *.Cu *.Mask F.SilkS))
+    (pad "" thru_hole circle (at 0 0) (size 4.064 4.064) (drill 3.048) (layers *.Cu *.Mask F.SilkS)
+      (net 84 "Net-(P11-Pad1)"))
   )
   (module Connect:1pin (layer F.Cu)
@@
     (descr "module 1 pin (ou trou mecanique de percage)")
     (tags DEV)
-    (fp_text reference REF** (at 0 -3.048) (layer F.SilkS) hide
-      (effects (font (size 1 1) (thickness 0.15)))
-    )
-    (fp_text value 1pin (at 0 2.794) (layer F.Fab) hide
+    (fp_text reference P12 (at 0 -3.048) (layer F.SilkS) hide
+      (effects (font (size 1 1) (thickness 0.15)))
+    )
+    (fp_text value CONN_1 (at 0 2.794) (layer F.Fab) hide
       (effects (font (size 1 1) (thickness 0.15)))
     )
     (fp_circle (center 0 0) (end 0 -2.286) (layer F.SilkS) (width 0.15))
-    (pad "" thru_hole circle (at 0 0) (size 4.064 4.064) (drill 3.048) (layers *.Cu *.Mask F.SilkS))
+    (pad "" thru_hole circle (at 0 0) (size 4.064 4.064) (drill 3.048) (layers *.Cu *.Mask F.SilkS)
+      (net 85 "Net-(P12-Pad1)"))
   )
   (module Connect:1pin (layer F.Cu)
@@
     (descr "module 1 pin (ou trou mecanique de percage)")
     (tags DEV)
-    (fp_text reference REF** (at 0 -3.048) (layer F.SilkS) hide
-      (effects (font (size 1 1) (thickness 0.15)))
-    )
-    (fp_text value 1pin (at 0 2.794) (layer F.Fab) hide
+    (fp_text reference P13 (at 0 -3.048) (layer F.SilkS) hide
+      (effects (font (size 1 1) (thickness 0.15)))
+    )
+    (fp_text value CONN_1 (at 0 2.794) (layer F.Fab) hide
       (effects (font (size 1 1) (thickness 0.15)))
     )
     (fp_circle (center 0 0) (end 0 -2.286) (layer F.SilkS) (width 0.15))
-    (pad "" thru_hole circle (at 0 0) (size 4.064 4.064) (drill 3.048) (layers *.Cu *.Mask F.SilkS))
-  )
-  (module Connect:1pin (layer F.Cu)
-    (at 199.898 119.126)
-    (descr "module 1 pin (ou trou mecanique de percage)")
-    (tags DEV)
-    (fp_text reference REF** (at 0 -3.048) (layer F.SilkS) hide
-      (effects (font (size 1 1) (thickness 0.15)))
-    )
-    (fp_text value 1pin (at 0 2.794) (layer F.Fab) hide
-      (effects (font (size 1 1) (thickness 0.15)))
-    )
-    (fp_circle (center 0 0) (end 0 -2.286) (layer F.SilkS) (width 0.15))
-    (pad "" thru_hole circle (at 0 0) (size 4.064 4.064) (drill 3.048) (layers *.Cu *.Mask F.SilkS))
-  )
-  (module Connect:1pin (layer F.Cu)
-    (at 169.418 114.046)
-    (descr "module 1 pin (ou trou mecanique de percage)")
-    (tags DEV)
-    (fp_text reference REF** (at 0 -3.048) (layer F.SilkS) hide
-      (effects (font (size 1 1) (thickness 0.15)))
-    )
-    (fp_text value 1pin (at 0 2.794) (layer F.Fab) hide
-      (effects (font (size 1 1) (thickness 0.15)))
-    )
-    (fp_circle (center 0 0) (end 0 -2.286) (layer F.SilkS) (width 0.15))
-    (pad "" thru_hole circle (at 0 0) (size 4.064 4.064) (drill 3.048) (layers *.Cu *.Mask F.SilkS))
-  )
-  (module Connect:1pin (layer F.Cu)
-    (at 117.348 119.126)
-    (descr "module 1 pin (ou trou mecanique de percage)")
-    (tags DEV)
-    (fp_text reference REF** (at 0 -3.048) (layer F.SilkS) hide
-      (effects (font (size 1 1) (thickness 0.15)))
-    )
-    (fp_text value 1pin (at 0 2.794) (layer F.Fab) hide
-      (effects (font (size 1 1) (thickness 0.15)))
-    )
-    (fp_circle (center 0 0) (end 0 -2.286) (layer F.SilkS) (width 0.15))
-    (pad "" thru_hole circle (at 0 0) (size 4.064 4.064) (drill 3.048) (layers *.Cu *.Mask F.SilkS))
+    (pad "" thru_hole circle (at 0 0) (size 4.064 4.064) (drill 3.048) (layers *.Cu *.Mask F.SilkS)
+      (net 86 "Net-(P13-Pad1)"))
   )
   (gr_line (start 175.6156 96.774) (end 175.6156 90.7288) (angle 90) (layer Dwgs.User) (width 0.15))

Commit message: corrections
Connections:
- net +3.3V renamed +3V3
- net /0(Rx) renamed /0(Rx0)
- net /1(Tx) renamed /1(Tx0)
- net /14(Tx) renamed /14(Tx3)
- net /15(Rx) renamed /15(Rx3)
- net /16(Tx) renamed /16(Tx2)
- net /17(Rx) renamed /17(Rx2)
- net /18(Tx) renamed /18(Tx1)
- net /19(Rx) renamed /19(Rx1)
- net /NC renamed Net-(P2-Pad1)
Other:
- board text added: "1"
