File: template/BeagleBone-Black-Cape/BeagleBone-Black-Cape.kicad_pcb (KiCad board)
At the start: 2 copper layers, 54.6 x 86.4 mm, 2 parts, among them P8 CONN_02X23, P9 CONN_02X23

Commit message: make 3d modules safe
Parts:
- P8, P9: value CONN_02X23 -> BeagleBone_Black_Header; footprint Pin_Headers:Pin_Header_Straight_2x23 -> Socket_BeagleBone_Black:Socket_BeagleBone_Black
Changed lines of the file:
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@@
-(kicad_pcb (version 4) (host pcbnew "(2015-06-23 BZR 5811)-product")
+(kicad_pcb (version 4) (host pcbnew "(2015-07-05 BZR 5886)-product")
   (general
     (links 10)
     (no_connects 10)
-    (area 114.463829 42.696129 169.076371 129.058671)
+    (area 106.333194 42.696129 174.667007 129.058671)
     (thickness 1.6)
     (drawings 11)
@@
     (mod_text_size 1 1)
     (mod_text_width 0.15)
-    (pad_size 1.5 1.5)
-    (pad_drill 0.6)
+    (pad_size 1.7272 1.7272)
+    (pad_drill 1.016)
     (pad_to_mask_clearance 0)
     (aux_axis_origin 0 0)
-    (visible_elements FFFFFF7F)
+    (visible_elements 7FFFFFFF)
     (pcbplotparams
       (layerselection 0x01030_80000001)
@@
     (add_net VDD_ADC)
   )
-  (module Pin_Headers:Pin_Header_Straight_2x23 locked (layer F.Cu)
+  (module Socket_BeagleBone_Black:Socket_BeagleBone_Black (layer F.Cu)
     (at 164.6301 62.3824)
     (descr "Through hole pin header")
@@
       (effects (font (size 1 1) (thickness 0.15)))
     )
-    (fp_text value CONN_02X23 (at 0 -3.1) (layer F.Fab)
+    (fp_text value BeagleBone_Black_Header (at 0 -3.1) (layer F.Fab)
       (effects (font (size 1 1) (thickness 0.15)))
     )
@@
     (pad 46 thru_hole oval (at 2.54 55.88) (size 1.7272 1.7272) (drill 1.016) (layers *.Cu *.Mask F.SilkS)
       (net 44 "Net-(P8-Pad46)"))
-    (model Pin_Headers.3dshapes/Pin_Header_Straight_2x23.wrl
-      (at (xyz 0.05 -1.1 -0.07000000000000001))
-      (scale (xyz 1 1 1))
-      (rotate (xyz 180 0 90))
-    )
-    (model Socket_Strips.3dshapes/Socket_Strip_Straight_2x23.wrl
+    (model ${KIPRJMOD}/Socket_BeagleBone_Black.3dshapes/Socket_BeagleBone_Black.wrl
       (at (xyz 0.05 -1.1 0))
       (scale (xyz 1 1 1))
@@
     )
   )
-  (module Pin_Headers:Pin_Header_Straight_2x23 locked (layer F.Cu)
+  (module Socket_BeagleBone_Black:Socket_BeagleBone_Black (layer F.Cu)
     (at 116.3701 62.3824)
     (descr "Through hole pin header")
@@
       (effects (font (size 1 1) (thickness 0.15)))
     )
-    (fp_text value CONN_02X23 (at 0 -3.1) (layer F.Fab)
+    (fp_text value BeagleBone_Black_Header (at 0 -3.1) (layer F.Fab)
       (effects (font (size 1 1) (thickness 0.15)))
     )
@@
     (pad 46 thru_hole oval (at 2.54 55.88) (size 1.7272 1.7272) (drill 1.016) (layers *.Cu *.Mask F.SilkS)
       (net 75 GNDD))
-    (model Pin_Headers.3dshapes/Pin_Header_Straight_2x23.wrl
-      (at (xyz 0.05 -1.1 -0.07000000000000001))
-      (scale (xyz 1 1 1))
-      (rotate (xyz 180 0 90))
-    )
-    (model Socket_Strips.3dshapes/Socket_Strip_Straight_2x23.wrl
+    (model ${KIPRJMOD}/Socket_BeagleBone_Black.3dshapes/Socket_BeagleBone_Black.wrl
       (at (xyz 0.05 -1.1 0))
       (scale (xyz 1 1 1))
