File: template/BeagleBone-Black-Cape/BeagleBone-Black-Cape.sch (KiCad schematic (older format))
At the start: 2 parts, among them P8 CONN_02X23, P9 CONN_02X23

Commit message: make 3d modules safe
Parts:
- removed P8, P9: CONN_02X23, Pin_Headers:Pin_Header_Straight_2x23, symbol CONN_02X23
- added P8, P9: BeagleBone_Black_Header, Socket_BeagleBone_Black:Socket_BeagleBone_Black, symbol BeagleBone_Black_Header
Changed lines of the file:
@@
 EESchema Schematic File Version 2
-LIBS:bbb-rescue
+LIBS:valves
 LIBS:power
 LIBS:device
@@
 LIBS:atmel
 LIBS:contrib
-LIBS:valves
-LIBS:bbb-cache
+LIBS:test-cache
 EELAYER 25 0
 EELAYER END
@@
 $EndDescr
 $Comp
-L CONN_02X23 P9
-U 1 1 5589720E
-P 2450 2250
-F 0 "P9" H 2450 3450 50  0000 C CNN
-F 1 "CONN_02X23" V 2450 2250 50  0000 C CNN
-F 2 "Pin_Headers:Pin_Header_Straight_2x23" H 2450 1400 60  0001 C CNN
-F 3 "" H 2450 1400 60  0000 C CNN
-	1    2450 2250
-	1    0    0    -1
-$EndComp
-$Comp
-L CONN_02X23 P8
-U 1 1 55897251
-P 5150 2250
-F 0 "P8" H 5150 3450 50  0000 C CNN
-F 1 "CONN_02X23" V 5150 2250 50  0000 C CNN
-F 2 "Pin_Headers:Pin_Header_Straight_2x23" H 5150 1400 60  0001 C CNN
-F 3 "" H 5150 1400 60  0000 C CNN
-	1    5150 2250
-	1    0    0    -1
-$EndComp
-$Comp
-L GNDD #PWR?
+L GNDD #PWR01
 U 1 1 5589785A
 P 2450 3650
-F 0 "#PWR?" H 2450 3400 50  0001 C CNN
+F 0 "#PWR01" H 2450 3400 50  0001 C CNN
 F 1 "GNDD" H 2450 3500 50  0000 C CNN
 F 2 "" H 2450 3650 60  0000 C CNN
@@
 Connection ~ 2450 3550
 $Comp
-L GNDD #PWR?
+L GNDD #PWR02
 U 1 1 558978D3
 P 3500 1150
-F 0 "#PWR?" H 3500 900 50  0001 C CNN
+F 0 "#PWR02" H 3500 900 50  0001 C CNN
 F 1 "GNDD" H 3500 1000 50  0000 C CNN
 F 2 "" H 3500 1150 60  0000 C CNN
@@
 $EndComp
 $Comp
-L GNDD #PWR?
+L GNDD #PWR03
 U 1 1 5589790A
 P 1400 1150
-F 0 "#PWR?" H 1400 900 50  0001 C CNN
+F 0 "#PWR03" H 1400 900 50  0001 C CNN
 F 1 "GNDD" H 1400 1000 50  0000 C CNN
 F 2 "" H 1400 1150 60  0000 C CNN
@@
 $EndComp
 $Comp
-L GNDD #PWR?
+L GNDD #PWR04
 U 1 1 558979C1
 P 4650 1150
-F 0 "#PWR?" H 4650 900 50  0001 C CNN
+F 0 "#PWR04" H 4650 900 50  0001 C CNN
 F 1 "GNDD" H 4650 1000 50  0000 C CNN
 F 2 "" H 4650 1150 60  0000 C CNN
@@
 $EndComp
 $Comp
-L GNDD #PWR?
+L GNDD #PWR05
 U 1 1 558979E8
 P 5650 1150
-F 0 "#PWR?" H 5650 900 50  0001 C CNN
+F 0 "#PWR05" H 5650 900 50  0001 C CNN
 F 1 "GNDD" H 5650 1000 50  0000 C CNN
 F 2 "" H 5650 1150 60  0000 C CNN
@@
 $EndComp
 $Comp
-L +3V3 #PWR?
+L +3V3 #PWR06
 U 1 1 55897A67
 P 2850 950
-F 0 "#PWR?" H 2850 800 50  0001 C CNN
+F 0 "#PWR06" H 2850 800 50  0001 C CNN
 F 1 "+3V3" H 2850 1090 50  0000 C CNN
 F 2 "" H 2850 950 60  0000 C CNN
@@
 $EndComp
 $Comp
-L +5V #PWR?
+L +5V #PWR07
 U 1 1 55897A7F
 P 3050 950
-F 0 "#PWR?" H 3050 800 50  0001 C CNN
+F 0 "#PWR07" H 3050 800 50  0001 C CNN
 F 1 "+5V" H 3050 1090 50  0000 C CNN
 F 2 "" H 3050 950 60  0000 C CNN
@@
 	3300 1450 2700 1450
 $Comp
-L +3V3 #PWR?
+L +3V3 #PWR08
 U 1 1 55897EE7
 P 2050 950
-F 0 "#PWR?" H 2050 800 50  0001 C CNN
+F 0 "#PWR08" H 2050 800 50  0001 C CNN
 F 1 "+3V3" H 2050 1090 50  0000 C CNN
 F 2 "" H 2050 950 60  0000 C CNN
@@
 $EndComp
 $Comp
-L +5V #PWR?
+L +5V #PWR09
 U 1 1 55897EF8
 P 1850 950
-F 0 "#PWR?" H 1850 800 50  0001 C CNN
+F 0 "#PWR09" H 1850 800 50  0001 C CNN
 F 1 "+5V" H 1850 1090 50  0000 C CNN
 F 2 "" H 1850 950 60  0000 C CNN
@@
 	5400 1150 5650 1150
 $Comp
-L SYS_5V #PWR?
+L SYS_5V #PWR010
 U 1 1 55898497
 P 3300 950
-F 0 "#PWR?" H 3300 800 50  0001 C CNN
+F 0 "#PWR010" H 3300 800 50  0001 C CNN
 F 1 "SYS_5V" H 3300 1090 50  0000 C CNN
 F 2 "" H 3300 950 60  0000 C CNN
@@
 $EndComp
 $Comp
-L SYS_5V #PWR?
+L SYS_5V #PWR011
 U 1 1 558984AF
 P 1600 950
-F 0 "#PWR?" H 1600 800 50  0001 C CNN
+F 0 "#PWR011" H 1600 800 50  0001 C CNN
 F 1 "SYS_5V" H 1600 1090 50  0000 C CNN
 F 2 "" H 1600 950 60  0000 C CNN
@@
 $EndComp
 $Comp
-L VDD_ADC #PWR?
+L VDD_ADC #PWR012
 U 1 1 558985D8
 P 3050 2550
-F 0 "#PWR?" H 3050 2400 50  0001 C CNN
+F 0 "#PWR012" H 3050 2400 50  0001 C CNN
 F 1 "VDD_ADC" H 3050 2690 50  0000 C CNN
 F 2 "" H 3050 2550 60  0000 C CNN
@@
 	3050 2650 3050 2550
 $Comp
-L GNDA_ADC #PWR?
+L GNDA_ADC #PWR013
 U 1 1 5589865D
 P 3050 2750
-F 0 "#PWR?" H 3050 2500 50  0001 C CNN
+F 0 "#PWR013" H 3050 2500 50  0001 C CNN
 F 1 "GNDA_ADC" H 3050 2600 50  0000 C CNN
 F 2 "" H 3050 2750 60  0000 C CNN
@@
 Wire Wire Line
 	2200 1550 2100 1550
+$Comp
+L BeagleBone_Black_Header P9
+U 1 1 55DF7DBA
+P 2450 2250
+F 0 "P9" H 2450 3450 50  0000 C CNN
+F 1 "BeagleBone_Black_Header" V 2450 2250 50  0000 C CNN
+F 2 "Socket_BeagleBone_Black:Socket_BeagleBone_Black" H 2450 1400 60  0001 C CNN
+F 3 "" H 2450 1400 60  0000 C CNN
+	1    2450 2250
+	1    0    0    -1
+$EndComp
+$Comp
+L BeagleBone_Black_Header P8
+U 1 1 55DF7DE1
+P 5150 2250
+F 0 "P8" H 5150 3450 50  0000 C CNN
+F 1 "BeagleBone_Black_Header" V 5150 2250 50  0000 C CNN
+F 2 "Socket_BeagleBone_Black:Socket_BeagleBone_Black" H 5150 1400 60  0001 C CNN
+F 3 "" H 5150 1400 60  0000 C CNN
+	1    5150 2250
+	1    0    0    -1
+$EndComp
 $EndSCHEMATC
