File: template/Arduino_Pro_Mini/Arduino_Pro_Mini.sch (KiCad schematic (older format))
At the start: 5 parts, among them P1 Digital, P2 COM, P3 ADC, P4 Analog, P5 ADC

Commit message: rebuilt shematic and fix librairie
Parts:
- removed P1: Digital, Socket_Arduino_Pro_Mini:Socket_Strip_Arduino_1x12, symbol CONN_12
- removed P2: COM, Socket_Arduino_Pro_Mini:Socket_Strip_Arduino_1x06, symbol CONN_6
- removed P3, P5: ADC, Socket_Arduino_Pro_Mini:Socket_Strip_Arduino_1x02, symbol CONN_2
- removed P4: Analog, Socket_Arduino_Pro_Mini:Socket_Strip_Arduino_1x12, symbol CONN_12
- added P1: Digital, Socket_Arduino_Pro_Mini:Socket_Strip_Arduino_1x12, symbol CONN_01X12
- added P2: COM, Socket_Arduino_Pro_Mini:Socket_Strip_Arduino_1x06, symbol CONN_01X06
- added P3, P5: ADC, Socket_Arduino_Pro_Mini:Socket_Strip_Arduino_1x02, symbol CONN_01X02
- added P4: Analog, Socket_Arduino_Pro_Mini:Socket_Strip_Arduino_1x12, symbol CONN_01X12
Connections:
- wire segments 40 -> 29
Other:
- note added: "1"
