File: template/Arduino_Fio/Arduino_Fio.kicad_pcb (KiCad board)
At the start: 2 copper layers, 27.9 x 64.8 mm, 2 parts, among them P1 Digital, P2 Analog

Commit message: rebuilt shematic and fix librairie
Connections:
- net +3.3V renamed +3V3
Changed lines of the file:
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@@
-(kicad_pcb (version 4) (host pcbnew "(2015-03-25 BZR 5536)-product")
+(kicad_pcb (version 4) (host pcbnew 4.0.2-4+6225~38~ubuntu14.04.1-stable)
   (general
     (links 2)
@@
   )
   (net 0 "")
-  (net 1 +3.3V)
-  (net 2 GND)
-  (net 3 /2)
-  (net 4 "/3(**)")
-  (net 5 /4)
-  (net 6 "/5(**)")
-  (net 7 "/6(**)")
-  (net 8 /7)
-  (net 9 /8)
-  (net 10 "/9(**)")
-  (net 11 "/10(**/SCK)")
-  (net 12 "/11(**/MOSI)")
-  (net 13 "/12(MISO)")
-  (net 14 "/13(SS)")
-  (net 15 /AREF)
-  (net 16 /RxI)
-  (net 17 /TxO)
-  (net 18 /DTR)
-  (net 19 /A0)
-  (net 20 /A1)
-  (net 21 /A2)
-  (net 22 /A3)
-  (net 23 "/A4(SDA)")
-  (net 24 "/A5(SCL)")
-  (net 25 /A6)
-  (net 26 /A7)
+  (net 1 GND)
+  (net 2 /2)
+  (net 3 "/3(**)")
+  (net 4 /4)
+  (net 5 "/5(**)")
+  (net 6 "/6(**)")
+  (net 7 /7)
+  (net 8 /8)
+  (net 9 "/9(**)")
+  (net 10 "/10(**/SCK)")
+  (net 11 "/11(**/MOSI)")
+  (net 12 "/12(MISO)")
+  (net 13 "/13(SS)")
+  (net 14 /AREF)
+  (net 15 /RxI)
+  (net 16 /TxO)
+  (net 17 /DTR)
+  (net 18 /A0)
+  (net 19 /A1)
+  (net 20 /A2)
+  (net 21 /A3)
+  (net 22 "/A4(SDA)")
+  (net 23 "/A5(SCL)")
+  (net 24 /A6)
+  (net 25 /A7)
+  (net 26 +3V3)
   (net_class Default "This is the default net class."
     (clearance 0.2)
@@
     (uvia_dia 0.3)
     (uvia_drill 0.1)
-    (add_net +3.3V)
+    (add_net +3V3)
     (add_net "/10(**/SCK)")
     (add_net "/11(**/MOSI)")
@@
     (fp_line (start 1.27 1.27) (end 1.27 -1.27) (layer F.SilkS) (width 0.15))
     (pad 1 thru_hole oval (at 0 0 270) (size 1.7272 2.032) (drill 1.016) (layers *.Cu *.Mask F.SilkS)
-      (net 1 +3.3V))
+      (net 26 +3V3))
     (pad 2 thru_hole oval (at 2.54 0 270) (size 1.7272 2.032) (drill 1.016) (layers *.Cu *.Mask F.SilkS)
-      (net 2 GND))
+      (net 1 GND))
     (pad 3 thru_hole oval (at 5.08 0 270) (size 1.7272 2.032) (drill 1.016) (layers *.Cu *.Mask F.SilkS)
-      (net 3 /2))
+      (net 2 /2))
     (pad 4 thru_hole oval (at 7.62 0 270) (size 1.7272 2.032) (drill 1.016) (layers *.Cu *.Mask F.SilkS)
-      (net 4 "/3(**)"))
+      (net 3 "/3(**)"))
     (pad 5 thru_hole oval (at 10.16 0 270) (size 1.7272 2.032) (drill 1.016) (layers *.Cu *.Mask F.SilkS)
-      (net 5 /4))
+      (net 4 /4))
     (pad 6 thru_hole oval (at 12.7 0 270) (size 1.7272 2.032) (drill 1.016) (layers *.Cu *.Mask F.SilkS)
-      (net 6 "/5(**)"))
+      (net 5 "/5(**)"))
     (pad 7 thru_hole oval (at 15.24 0 270) (size 1.7272 2.032) (drill 1.016) (layers *.Cu *.Mask F.SilkS)
-      (net 7 "/6(**)"))
+      (net 6 "/6(**)"))
     (pad 8 thru_hole oval (at 17.78 0 270) (size 1.7272 2.032) (drill 1.016) (layers *.Cu *.Mask F.SilkS)
-      (net 8 /7))
+      (net 7 /7))
     (pad 9 thru_hole oval (at 20.32 0 270) (size 1.7272 2.032) (drill 1.016) (layers *.Cu *.Mask F.SilkS)
-      (net 9 /8))
+      (net 8 /8))
     (pad 10 thru_hole oval (at 22.86 0 270) (size 1.7272 2.032) (drill 1.016) (layers *.Cu *.Mask F.SilkS)
-      (net 10 "/9(**)"))
+      (net 9 "/9(**)"))
     (pad 11 thru_hole oval (at 25.4 0 270) (size 1.7272 2.032) (drill 1.016) (layers *.Cu *.Mask F.SilkS)
-      (net 11 "/10(**/SCK)"))
+      (net 10 "/10(**/SCK)"))
     (pad 12 thru_hole oval (at 27.94 0 270) (size 1.7272 2.032) (drill 1.016) (layers *.Cu *.Mask F.SilkS)
-      (net 12 "/11(**/MOSI)"))
+      (net 11 "/11(**/MOSI)"))
     (pad 13 thru_hole oval (at 30.48 0 270) (size 1.7272 2.032) (drill 1.016) (layers *.Cu *.Mask F.SilkS)
-      (net 13 "/12(MISO)"))
+      (net 12 "/12(MISO)"))
     (pad 14 thru_hole oval (at 33.02 0 270) (size 1.7272 2.032) (drill 1.016) (layers *.Cu *.Mask F.SilkS)
-      (net 14 "/13(SS)"))
+      (net 13 "/13(SS)"))
     (model ${KIPRJMOD}/Socket_Arduino_Fio.3dshapes/Socket_header_Arduino_1x14.wrl
       (at (xyz 0.65 0 0))
@@
     (fp_line (start 1.27 1.27) (end 1.27 -1.27) (layer F.SilkS) (width 0.15))
     (pad 1 thru_hole oval (at 0 0 270) (size 1.7272 2.032) (drill 1.016) (layers *.Cu *.Mask F.SilkS)
-      (net 2 GND))
+      (net 1 GND))
     (pad 2 thru_hole oval (at 2.54 0 270) (size 1.7272 2.032) (drill 1.016) (layers *.Cu *.Mask F.SilkS)
-      (net 15 /AREF))
+      (net 14 /AREF))
     (pad 3 thru_hole oval (at 5.08 0 270) (size 1.7272 2.032) (drill 1.016) (layers *.Cu *.Mask F.SilkS)
-      (net 1 +3.3V))
+      (net 26 +3V3))
     (pad 4 thru_hole oval (at 7.62 0 270) (size 1.7272 2.032) (drill 1.016) (layers *.Cu *.Mask F.SilkS)
-      (net 16 /RxI))
+      (net 15 /RxI))
     (pad 5 thru_hole oval (at 10.16 0 270) (size 1.7272 2.032) (drill 1.016) (layers *.Cu *.Mask F.SilkS)
-      (net 17 /TxO))
+      (net 16 /TxO))
     (pad 6 thru_hole oval (at 12.7 0 270) (size 1.7272 2.032) (drill 1.016) (layers *.Cu *.Mask F.SilkS)
-      (net 18 /DTR))
+      (net 17 /DTR))
     (pad 7 thru_hole oval (at 15.24 0 270) (size 1.7272 2.032) (drill 1.016) (layers *.Cu *.Mask F.SilkS)
-      (net 19 /A0))
+      (net 18 /A0))
     (pad 8 thru_hole oval (at 17.78 0 270) (size 1.7272 2.032) (drill 1.016) (layers *.Cu *.Mask F.SilkS)
-      (net 20 /A1))
+      (net 19 /A1))
     (pad 9 thru_hole oval (at 20.32 0 270) (size 1.7272 2.032) (drill 1.016) (layers *.Cu *.Mask F.SilkS)
-      (net 21 /A2))
+      (net 20 /A2))
     (pad 10 thru_hole oval (at 22.86 0 270) (size 1.7272 2.032) (drill 1.016) (layers *.Cu *.Mask F.SilkS)
-      (net 22 /A3))
+      (net 21 /A3))
     (pad 11 thru_hole oval (at 25.4 0 270) (size 1.7272 2.032) (drill 1.016) (layers *.Cu *.Mask F.SilkS)
-      (net 23 "/A4(SDA)"))
+      (net 22 "/A4(SDA)"))
     (pad 12 thru_hole oval (at 27.94 0 270) (size 1.7272 2.032) (drill 1.016) (layers *.Cu *.Mask F.SilkS)
-      (net 24 "/A5(SCL)"))
+      (net 23 "/A5(SCL)"))
     (pad 13 thru_hole oval (at 30.48 0 270) (size 1.7272 2.032) (drill 1.016) (layers *.Cu *.Mask F.SilkS)
-      (net 25 /A6))
+      (net 24 /A6))
     (pad 14 thru_hole oval (at 33.02 0 270) (size 1.7272 2.032) (drill 1.016) (layers *.Cu *.Mask F.SilkS)
-      (net 26 /A7))
+      (net 25 /A7))
     (model ${KIPRJMOD}/Socket_Arduino_Fio.3dshapes/Socket_header_Arduino_1x14.wrl
       (at (xyz 0.65 0 0))

Commit message: Fix pin order SS, MOSI, MISO, SCK
Connections:
- net /10(**/SCK) renamed /10(**/SS)
- net /13(SS) renamed /13(SCK)
Changed lines of the file:
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@@
-(kicad_pcb (version 4) (host pcbnew 4.0.2-4+6225~38~ubuntu14.04.1-stable)
+(kicad_pcb (version 4) (host pcbnew 4.0.4+e1-6308~48~ubuntu14.04.1-stable)
   (general
     (links 2)
@@
   (net 8 /8)
   (net 9 "/9(**)")
-  (net 10 "/10(**/SCK)")
-  (net 11 "/11(**/MOSI)")
-  (net 12 "/12(MISO)")
-  (net 13 "/13(SS)")
-  (net 14 /AREF)
-  (net 15 /RxI)
-  (net 16 /TxO)
-  (net 17 /DTR)
-  (net 18 /A0)
-  (net 19 /A1)
-  (net 20 /A2)
-  (net 21 /A3)
-  (net 22 "/A4(SDA)")
-  (net 23 "/A5(SCL)")
-  (net 24 /A6)
-  (net 25 /A7)
-  (net 26 +3V3)
+  (net 10 "/11(**/MOSI)")
+  (net 11 "/12(MISO)")
+  (net 12 /AREF)
+  (net 13 /RxI)
+  (net 14 /TxO)
+  (net 15 /DTR)
+  (net 16 /A0)
+  (net 17 /A1)
+  (net 18 /A2)
+  (net 19 /A3)
+  (net 20 "/A4(SDA)")
+  (net 21 "/A5(SCL)")
+  (net 22 /A6)
+  (net 23 /A7)
+  (net 24 +3V3)
+  (net 25 "/10(**/SS)")
+  (net 26 "/13(SCK)")
   (net_class Default "This is the default net class."
     (clearance 0.2)
@@
     (uvia_drill 0.1)
     (add_net +3V3)
-    (add_net "/10(**/SCK)")
+    (add_net "/10(**/SS)")
     (add_net "/11(**/MOSI)")
     (add_net "/12(MISO)")
-    (add_net "/13(SS)")
+    (add_net "/13(SCK)")
     (add_net /2)
     (add_net "/3(**)")
@@
     (fp_line (start 1.27 1.27) (end 1.27 -1.27) (layer F.SilkS) (width 0.15))
     (pad 1 thru_hole oval (at 0 0 270) (size 1.7272 2.032) (drill 1.016) (layers *.Cu *.Mask F.SilkS)
-      (net 26 +3V3))
+      (net 24 +3V3))
     (pad 2 thru_hole oval (at 2.54 0 270) (size 1.7272 2.032) (drill 1.016) (layers *.Cu *.Mask F.SilkS)
       (net 1 GND))
@@
       (net 9 "/9(**)"))
     (pad 11 thru_hole oval (at 25.4 0 270) (size 1.7272 2.032) (drill 1.016) (layers *.Cu *.Mask F.SilkS)
-      (net 10 "/10(**/SCK)"))
+      (net 25 "/10(**/SS)"))
     (pad 12 thru_hole oval (at 27.94 0 270) (size 1.7272 2.032) (drill 1.016) (layers *.Cu *.Mask F.SilkS)
-      (net 11 "/11(**/MOSI)"))
+      (net 10 "/11(**/MOSI)"))
     (pad 13 thru_hole oval (at 30.48 0 270) (size 1.7272 2.032) (drill 1.016) (layers *.Cu *.Mask F.SilkS)
-      (net 12 "/12(MISO)"))
+      (net 11 "/12(MISO)"))
     (pad 14 thru_hole oval (at 33.02 0 270) (size 1.7272 2.032) (drill 1.016) (layers *.Cu *.Mask F.SilkS)
-      (net 13 "/13(SS)"))
+      (net 26 "/13(SCK)"))
     (model ${KIPRJMOD}/Socket_Arduino_Fio.3dshapes/Socket_header_Arduino_1x14.wrl
       (at (xyz 0.65 0 0))
@@
       (net 1 GND))
     (pad 2 thru_hole oval (at 2.54 0 270) (size 1.7272 2.032) (drill 1.016) (layers *.Cu *.Mask F.SilkS)
-      (net 14 /AREF))
+      (net 12 /AREF))
     (pad 3 thru_hole oval (at 5.08 0 270) (size 1.7272 2.032) (drill 1.016) (layers *.Cu *.Mask F.SilkS)
-      (net 26 +3V3))
+      (net 24 +3V3))
     (pad 4 thru_hole oval (at 7.62 0 270) (size 1.7272 2.032) (drill 1.016) (layers *.Cu *.Mask F.SilkS)
-      (net 15 /RxI))
+      (net 13 /RxI))
     (pad 5 thru_hole oval (at 10.16 0 270) (size 1.7272 2.032) (drill 1.016) (layers *.Cu *.Mask F.SilkS)
-      (net 16 /TxO))
+      (net 14 /TxO))
     (pad 6 thru_hole oval (at 12.7 0 270) (size 1.7272 2.032) (drill 1.016) (layers *.Cu *.Mask F.SilkS)
-      (net 17 /DTR))
+      (net 15 /DTR))
     (pad 7 thru_hole oval (at 15.24 0 270) (size 1.7272 2.032) (drill 1.016) (layers *.Cu *.Mask F.SilkS)
-      (net 18 /A0))
+      (net 16 /A0))
     (pad 8 thru_hole oval (at 17.78 0 270) (size 1.7272 2.032) (drill 1.016) (layers *.Cu *.Mask F.SilkS)
-      (net 19 /A1))
+      (net 17 /A1))
     (pad 9 thru_hole oval (at 20.32 0 270) (size 1.7272 2.032) (drill 1.016) (layers *.Cu *.Mask F.SilkS)
-      (net 20 /A2))
+      (net 18 /A2))
     (pad 10 thru_hole oval (at 22.86 0 270) (size 1.7272 2.032) (drill 1.016) (layers *.Cu *.Mask F.SilkS)
-      (net 21 /A3))
+      (net 19 /A3))
     (pad 11 thru_hole oval (at 25.4 0 270) (size 1.7272 2.032) (drill 1.016) (layers *.Cu *.Mask F.SilkS)
-      (net 22 "/A4(SDA)"))
+      (net 20 "/A4(SDA)"))
     (pad 12 thru_hole oval (at 27.94 0 270) (size 1.7272 2.032) (drill 1.016) (layers *.Cu *.Mask F.SilkS)
-      (net 23 "/A5(SCL)"))
+      (net 21 "/A5(SCL)"))
     (pad 13 thru_hole oval (at 30.48 0 270) (size 1.7272 2.032) (drill 1.016) (layers *.Cu *.Mask F.SilkS)
-      (net 24 /A6))
+      (net 22 /A6))
     (pad 14 thru_hole oval (at 33.02 0 270) (size 1.7272 2.032) (drill 1.016) (layers *.Cu *.Mask F.SilkS)
-      (net 25 /A7))
+      (net 23 /A7))
     (model ${KIPRJMOD}/Socket_Arduino_Fio.3dshapes/Socket_header_Arduino_1x14.wrl
       (at (xyz 0.65 0 0))
