File: template/Arduino_Nano/Arduino_Nano.kicad_pcb (KiCad board)
At the start: 2 copper layers, 17.8 x 43.2 mm, 6 parts, among them P1 Digital, P2 Analog, P3 CONN_1, P4 CONN_1, P5 CONN_1, P6 CONN_1

Commit message: rebuilt shematic and fix librairie
Parts:
- P3, P4, P5, P6: value CONN_1 -> CONN_01X01
Connections:
- net +3.3V renamed +3V3
Changed lines of the file:
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@@
-(kicad_pcb (version 4) (host pcbnew "(2015-03-25 BZR 5536)-product")
+(kicad_pcb (version 4) (host pcbnew 4.0.2-4+6225~38~ubuntu14.04.1-stable)
   (general
     (links 2)
     (no_connects 2)
-    (area 136.242429 65.55 157.889572 112.597001)
+    (area 138.125999 67.386999 156.006001 110.667001)
     (thickness 1.6)
     (drawings 20)
@@
   (net 25 /A0)
   (net 26 /AREF)
-  (net 27 +3.3V)
-  (net 28 "/13(SCK)")
-  (net 29 "Net-(P3-Pad1)")
-  (net 30 "Net-(P4-Pad1)")
-  (net 31 "Net-(P5-Pad1)")
-  (net 32 "Net-(P6-Pad1)")
+  (net 27 "/13(SCK)")
+  (net 28 "Net-(P3-Pad1)")
+  (net 29 "Net-(P4-Pad1)")
+  (net 30 "Net-(P5-Pad1)")
+  (net 31 "Net-(P6-Pad1)")
+  (net 32 +3V3)
   (net_class Default "This is the default net class."
     (clearance 0.2)
@@
     (uvia_dia 0.3)
     (uvia_drill 0.1)
-    (add_net +3.3V)
+    (add_net +3V3)
     (add_net +5V)
     (add_net "/0(Rx)")
@@
       (net 26 /AREF))
     (pad 14 thru_hole oval (at 33.02 0 270) (size 1.7272 2.032) (drill 1.016) (layers *.Cu *.Mask F.SilkS)
-      (net 27 +3.3V))
+      (net 32 +3V3))
     (pad 15 thru_hole oval (at 35.56 0 270) (size 1.7272 2.032) (drill 1.016) (layers *.Cu *.Mask F.SilkS)
-      (net 28 "/13(SCK)"))
+      (net 27 "/13(SCK)"))
     (model ${KIPRJMOD}/Socket_Arduino_Nano.3dshapes/Socket_header_Arduino_1x15.wrl
       (at (xyz 0.7 0 0))
@@
       (effects (font (size 1 1) (thickness 0.15)))
     )
-    (fp_text value CONN_1 (at 0 2.032) (layer F.Fab) hide
+    (fp_text value CONN_01X01 (at 0 2.032) (layer F.Fab) hide
       (effects (font (size 1 1) (thickness 0.15)))
     )
     (pad 1 thru_hole circle (at 0 0) (size 2.54 2.54) (drill 1.778) (layers *.Cu *.Mask F.SilkS)
-      (net 29 "Net-(P3-Pad1)"))
+      (net 28 "Net-(P3-Pad1)"))
   )
   (module Socket_Arduino_Nano:1pin_Nano locked (layer F.Cu)
@@
       (effects (font (size 1 1) (thickness 0.15)))
     )
-    (fp_text value CONN_1 (at 0 2.032) (layer F.Fab) hide
+    (fp_text value CONN_01X01 (at 0 2.032) (layer F.Fab) hide
       (effects (font (size 1 1) (thickness 0.15)))
     )
     (pad 1 thru_hole circle (at 0 0) (size 2.54 2.54) (drill 1.778) (layers *.Cu *.Mask F.SilkS)
-      (net 30 "Net-(P4-Pad1)"))
+      (net 29 "Net-(P4-Pad1)"))
   )
   (module Socket_Arduino_Nano:1pin_Nano locked (layer F.Cu)
@@
       (effects (font (size 1 1) (thickness 0.15)))
     )
-    (fp_text value CONN_1 (at 0 2.032) (layer F.Fab) hide
+    (fp_text value CONN_01X01 (at 0 2.032) (layer F.Fab) hide
       (effects (font (size 1 1) (thickness 0.15)))
     )
     (pad 1 thru_hole circle (at 0 0) (size 2.54 2.54) (drill 1.778) (layers *.Cu *.Mask F.SilkS)
-      (net 31 "Net-(P5-Pad1)"))
+      (net 30 "Net-(P5-Pad1)"))
   )
   (module Socket_Arduino_Nano:1pin_Nano locked (layer F.Cu)
@@
       (effects (font (size 1 1) (thickness 0.15)))
     )
-    (fp_text value CONN_1 (at 0 2.032) (layer F.Fab) hide
+    (fp_text value CONN_01X01 (at 0 2.032) (layer F.Fab) hide
       (effects (font (size 1 1) (thickness 0.15)))
     )
     (pad 1 thru_hole circle (at 0 0) (size 2.54 2.54) (drill 1.778) (layers *.Cu *.Mask F.SilkS)
-      (net 32 "Net-(P6-Pad1)"))
+      (net 31 "Net-(P6-Pad1)"))
   )
   (gr_text 1 (at 141.732 71.247) (layer F.SilkS)

Commit message: Fix pin order SS, MOSI, MISO, SCK
Connections:
- net /11(**/MISO) renamed /11(**/MOSI)
- net /12(MOSI) renamed /12(MISO)
Changed lines of the file:
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@@
-(kicad_pcb (version 4) (host pcbnew 4.0.2-4+6225~38~ubuntu14.04.1-stable)
+(kicad_pcb (version 4) (host pcbnew 4.0.4+e1-6308~48~ubuntu14.04.1-stable)
   (general
     (links 2)
@@
   (net 12 "/9(**)")
   (net 13 "/10(**/SS)")
-  (net 14 "/11(**/MISO)")
-  (net 15 "/12(MOSI)")
-  (net 16 /Vin)
-  (net 17 +5V)
-  (net 18 /A7)
-  (net 19 /A6)
-  (net 20 /A5)
-  (net 21 /A4)
-  (net 22 /A3)
-  (net 23 /A2)
-  (net 24 /A1)
-  (net 25 /A0)
-  (net 26 /AREF)
-  (net 27 "/13(SCK)")
-  (net 28 "Net-(P3-Pad1)")
-  (net 29 "Net-(P4-Pad1)")
-  (net 30 "Net-(P5-Pad1)")
-  (net 31 "Net-(P6-Pad1)")
-  (net 32 +3V3)
+  (net 14 /Vin)
+  (net 15 +5V)
+  (net 16 /A7)
+  (net 17 /A6)
+  (net 18 /A5)
+  (net 19 /A4)
+  (net 20 /A3)
+  (net 21 /A2)
+  (net 22 /A1)
+  (net 23 /A0)
+  (net 24 /AREF)
+  (net 25 "/13(SCK)")
+  (net 26 "Net-(P3-Pad1)")
+  (net 27 "Net-(P4-Pad1)")
+  (net 28 "Net-(P5-Pad1)")
+  (net 29 "Net-(P6-Pad1)")
+  (net 30 +3V3)
+  (net 31 "/11(**/MOSI)")
+  (net 32 "/12(MISO)")
   (net_class Default "This is the default net class."
     (clearance 0.2)
@@
     (add_net "/1(Tx)")
     (add_net "/10(**/SS)")
-    (add_net "/11(**/MISO)")
-    (add_net "/12(MOSI)")
+    (add_net "/11(**/MOSI)")
+    (add_net "/12(MISO)")
     (add_net "/13(SCK)")
     (add_net /2)
@@
       (net 13 "/10(**/SS)"))
     (pad 14 thru_hole oval (at 33.02 0 270) (size 1.7272 2.032) (drill 1.016) (layers *.Cu *.Mask F.SilkS)
-      (net 14 "/11(**/MISO)"))
+      (net 31 "/11(**/MOSI)"))
     (pad 15 thru_hole oval (at 35.56 0 270) (size 1.7272 2.032) (drill 1.016) (layers *.Cu *.Mask F.SilkS)
-      (net 15 "/12(MOSI)"))
+      (net 32 "/12(MISO)"))
     (model ${KIPRJMOD}/Socket_Arduino_Nano.3dshapes/Socket_header_Arduino_1x15.wrl
       (at (xyz 0.7 0 0))
@@
     (fp_line (start 1.27 1.27) (end 1.27 -1.27) (layer F.SilkS) (width 0.15))
     (pad 1 thru_hole oval (at 0 0 270) (size 1.7272 2.032) (drill 1.016) (layers *.Cu *.Mask F.SilkS)
-      (net 16 /Vin))
+      (net 14 /Vin))
     (pad 2 thru_hole oval (at 2.54 0 270) (size 1.7272 2.032) (drill 1.016) (layers *.Cu *.Mask F.SilkS)
       (net 4 GND))
@@
       (net 3 /Reset))
     (pad 4 thru_hole oval (at 7.62 0 270) (size 1.7272 2.032) (drill 1.016) (layers *.Cu *.Mask F.SilkS)
-      (net 17 +5V))
+      (net 15 +5V))
     (pad 5 thru_hole oval (at 10.16 0 270) (size 1.7272 2.032) (drill 1.016) (layers *.Cu *.Mask F.SilkS)
-      (net 18 /A7))
+      (net 16 /A7))
     (pad 6 thru_hole oval (at 12.7 0 270) (size 1.7272 2.032) (drill 1.016) (layers *.Cu *.Mask F.SilkS)
-      (net 19 /A6))
+      (net 17 /A6))
     (pad 7 thru_hole oval (at 15.24 0 270) (size 1.7272 2.032) (drill 1.016) (layers *.Cu *.Mask F.SilkS)
-      (net 20 /A5))
+      (net 18 /A5))
     (pad 8 thru_hole oval (at 17.78 0 270) (size 1.7272 2.032) (drill 1.016) (layers *.Cu *.Mask F.SilkS)
-      (net 21 /A4))
+      (net 19 /A4))
     (pad 9 thru_hole oval (at 20.32 0 270) (size 1.7272 2.032) (drill 1.016) (layers *.Cu *.Mask F.SilkS)
-      (net 22 /A3))
+      (net 20 /A3))
     (pad 10 thru_hole oval (at 22.86 0 270) (size 1.7272 2.032) (drill 1.016) (layers *.Cu *.Mask F.SilkS)
-      (net 23 /A2))
+      (net 21 /A2))
     (pad 11 thru_hole oval (at 25.4 0 270) (size 1.7272 2.032) (drill 1.016) (layers *.Cu *.Mask F.SilkS)
-      (net 24 /A1))
+      (net 22 /A1))
     (pad 12 thru_hole oval (at 27.94 0 270) (size 1.7272 2.032) (drill 1.016) (layers *.Cu *.Mask F.SilkS)
-      (net 25 /A0))
+      (net 23 /A0))
     (pad 13 thru_hole oval (at 30.48 0 270) (size 1.7272 2.032) (drill 1.016) (layers *.Cu *.Mask F.SilkS)
-      (net 26 /AREF))
+      (net 24 /AREF))
     (pad 14 thru_hole oval (at 33.02 0 270) (size 1.7272 2.032) (drill 1.016) (layers *.Cu *.Mask F.SilkS)
-      (net 32 +3V3))
+      (net 30 +3V3))
     (pad 15 thru_hole oval (at 35.56 0 270) (size 1.7272 2.032) (drill 1.016) (layers *.Cu *.Mask F.SilkS)
-      (net 27 "/13(SCK)"))
+      (net 25 "/13(SCK)"))
     (model ${KIPRJMOD}/Socket_Arduino_Nano.3dshapes/Socket_header_Arduino_1x15.wrl
       (at (xyz 0.7 0 0))
@@
     )
     (pad 1 thru_hole circle (at 0 0) (size 2.54 2.54) (drill 1.778) (layers *.Cu *.Mask F.SilkS)
-      (net 28 "Net-(P3-Pad1)"))
+      (net 26 "Net-(P3-Pad1)"))
   )
   (module Socket_Arduino_Nano:1pin_Nano locked (layer F.Cu)
@@
     )
     (pad 1 thru_hole circle (at 0 0) (size 2.54 2.54) (drill 1.778) (layers *.Cu *.Mask F.SilkS)
-      (net 29 "Net-(P4-Pad1)"))
+      (net 27 "Net-(P4-Pad1)"))
   )
   (module Socket_Arduino_Nano:1pin_Nano locked (layer F.Cu)
@@
     )
     (pad 1 thru_hole circle (at 0 0) (size 2.54 2.54) (drill 1.778) (layers *.Cu *.Mask F.SilkS)
-      (net 30 "Net-(P5-Pad1)"))
+      (net 28 "Net-(P5-Pad1)"))
   )
   (module Socket_Arduino_Nano:1pin_Nano locked (layer F.Cu)
@@
     )
     (pad 1 thru_hole circle (at 0 0) (size 2.54 2.54) (drill 1.778) (layers *.Cu *.Mask F.SilkS)
-      (net 31 "Net-(P6-Pad1)"))
+      (net 29 "Net-(P6-Pad1)"))
   )
   (gr_text 1 (at 141.732 71.247) (layer F.SilkS)
