File: template/Arduino_Mini/Arduino_Mini.kicad_pcb (KiCad board)
At the start: 2 copper layers, 17.8 x 30.5 mm, 6 parts, among them P1 ADC, P2 Digital, P3 ADC, P4 COM, P5 Analog, P6 PWR

Commit message: Fix pin order SS, MOSI, MISO, SCK
Connections:
- net /11(MISO) renamed /11(MOSI)
- net /12(**/MOSI) renamed /12(**/MISO)
Changed lines of the file:
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@@
-(kicad_pcb (version 4) (host pcbnew 4.0.2-4+6225~38~ubuntu14.04.1-stable)
+(kicad_pcb (version 4) (host pcbnew 4.0.4+e1-6308~48~ubuntu14.04.1-stable)
   (general
     (links 9)
@@
   (net 22 /A0)
   (net 23 "/13(SCK)")
-  (net 24 "/12(**/MOSI)")
-  (net 25 "/11(MISO)")
-  (net 26 "/10(**/SS)")
+  (net 24 "/10(**/SS)")
+  (net 25 "/12(**/MISO)")
+  (net 26 "/11(MOSI)")
   (net_class Default "This is the default net class."
     (clearance 0.2)
@@
     (add_net "/1(Tx)")
     (add_net "/10(**/SS)")
-    (add_net "/11(MISO)")
-    (add_net "/12(**/MOSI)")
+    (add_net "/11(MOSI)")
+    (add_net "/12(**/MISO)")
     (add_net "/13(SCK)")
     (add_net /2)
@@
       (net 23 "/13(SCK)"))
     (pad 10 thru_hole oval (at 22.86 0 270) (size 1.7272 2.032) (drill 1.016) (layers *.Cu *.Mask F.SilkS)
-      (net 24 "/12(**/MOSI)"))
+      (net 25 "/12(**/MISO)"))
     (pad 11 thru_hole oval (at 25.4 0 270) (size 1.7272 2.032) (drill 1.016) (layers *.Cu *.Mask F.SilkS)
-      (net 25 "/11(MISO)"))
+      (net 26 "/11(MOSI)"))
     (pad 12 thru_hole oval (at 27.94 0 270) (size 1.7272 2.032) (drill 1.016) (layers *.Cu *.Mask F.SilkS)
-      (net 26 "/10(**/SS)"))
+      (net 24 "/10(**/SS)"))
     (model ${KIPRJMOD}/Socket_Arduino_Mini.3dshapes/Socket_header_Arduino_1x12.wrl
       (at (xyz 0.55 0 0))

Commit message: On Template Arduino_Mini change connector P4 pin 1 : rst to 7
Connections:
- P4 pad 1: /Reset -> /7
Changed lines of the file:
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@@
-(kicad_pcb (version 4) (host pcbnew 4.0.4+e1-6308~48~ubuntu14.04.1-stable)
+(kicad_pcb (version 4) (host pcbnew 4.0.5-e0-6337~49~ubuntu14.04.1)
   (general
     (links 9)
@@
     (fp_line (start 1.27 1.27) (end 1.27 -1.27) (layer F.SilkS) (width 0.15))
     (pad 1 thru_hole oval (at 0 0) (size 1.7272 2.032) (drill 1.016) (layers *.Cu *.Mask F.SilkS)
-      (net 5 /Reset))
+      (net 12 /7))
     (pad 2 thru_hole oval (at 2.54 0) (size 1.7272 2.032) (drill 1.016) (layers *.Cu *.Mask F.SilkS)
       (net 3 "/1(Tx)"))
