File: template/Microduino_Core/Microduino_Core.kicad_pcb (KiCad board)
At the start: 2 copper layers, 27.9 x 25.4 mm, 1 part, among them U1 Microduino-Core

Commit message: last small changes
Parts:
- U1: footprint microduino:Microduino-27upin -> Modules:Microduino-27upin
Changed lines of the file:
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@@
-(kicad_pcb (version 4) (host pcbnew 4.0.2+dfsg1-stable)
+(kicad_pcb (version 4) (host pcbnew 4.0.7-e2-6376~58~ubuntu16.04.1)
   (general
     (links 0)
@@
     (mod_text_size 1 1)
     (mod_text_width 0.15)
-    (pad_size 2.032 2.032)
-    (pad_drill 1.016)
+    (pad_size 1.524 1.524)
+    (pad_drill 0.762)
     (pad_to_mask_clearance 0.2)
     (aux_axis_origin 0 0)
@@
     (uvia_drill 0.1)
   )
-  (module microduino:Microduino-27upin (layer F.Cu)
+  (module Modules:Microduino-27upin (layer F.Cu)
     (at 162.56 127 90)
-    (descr 15)
+    (descr 6)
     (fp_text reference U1 (at 12.7 -12.7 90) (layer F.SilkS)
       (effects (font (size 1 1) (thickness 0.15)))
@@
     (fp_line (start 24.13 -1.27) (end 1.27 -1.27) (layer F.SilkS) (width 0.15))
     (fp_line (start 1.27 -1.27) (end 1.27 -26.67) (layer F.SilkS) (width 0.15))
-    (pad 19 thru_hole circle (at 2.54 -5.08 90) (size 1.524 1.524) (drill 0.762) (layers *.Cu *.Mask F.SilkS))
-    (pad 20 thru_hole circle (at 2.54 -7.62 90) (size 1.524 1.524) (drill 0.762) (layers *.Cu *.Mask F.SilkS))
-    (pad 21 thru_hole circle (at 2.54 -10.16 90) (size 1.524 1.524) (drill 0.762) (layers *.Cu *.Mask F.SilkS))
-    (pad 22 thru_hole circle (at 2.54 -12.7 90) (size 1.524 1.524) (drill 0.762) (layers *.Cu *.Mask F.SilkS))
-    (pad 23 thru_hole circle (at 2.54 -15.24 90) (size 1.524 1.524) (drill 0.762) (layers *.Cu *.Mask F.SilkS))
-    (pad 24 thru_hole circle (at 2.54 -17.78 90) (size 1.524 1.524) (drill 0.762) (layers *.Cu *.Mask F.SilkS))
-    (pad 25 thru_hole circle (at 2.54 -20.32 90) (size 1.524 1.524) (drill 0.762) (layers *.Cu *.Mask F.SilkS))
-    (pad 26 thru_hole circle (at 2.54 -22.86 90) (size 1.524 1.524) (drill 0.762) (layers *.Cu *.Mask F.SilkS))
-    (pad 27 thru_hole circle (at 2.54 -25.4 90) (size 1.524 1.524) (drill 0.762) (layers *.Cu *.Mask F.SilkS))
-    (pad 18 thru_hole circle (at 2.54 -2.54 90) (size 1.524 1.524) (drill 0.762) (layers *.Cu *.Mask F.SilkS))
-    (pad 17 thru_hole circle (at 5.08 -2.54 90) (size 1.524 1.524) (drill 0.762) (layers *.Cu *.Mask F.SilkS))
-    (pad 16 thru_hole circle (at 7.62 -2.54 90) (size 1.524 1.524) (drill 0.762) (layers *.Cu *.Mask F.SilkS))
-    (pad 15 thru_hole circle (at 10.16 -2.54 90) (size 1.524 1.524) (drill 0.762) (layers *.Cu *.Mask F.SilkS))
+    (pad 9 thru_hole circle (at 2.54 -5.08 90) (size 1.524 1.524) (drill 0.762) (layers *.Cu *.Mask F.SilkS))
+    (pad 8 thru_hole circle (at 2.54 -7.62 90) (size 1.524 1.524) (drill 0.762) (layers *.Cu *.Mask F.SilkS))
+    (pad 7 thru_hole circle (at 2.54 -10.16 90) (size 1.524 1.524) (drill 0.762) (layers *.Cu *.Mask F.SilkS))
+    (pad 6 thru_hole circle (at 2.54 -12.7 90) (size 1.524 1.524) (drill 0.762) (layers *.Cu *.Mask F.SilkS))
+    (pad 5 thru_hole circle (at 2.54 -15.24 90) (size 1.524 1.524) (drill 0.762) (layers *.Cu *.Mask F.SilkS))
+    (pad 4 thru_hole circle (at 2.54 -17.78 90) (size 1.524 1.524) (drill 0.762) (layers *.Cu *.Mask F.SilkS))
+    (pad 3 thru_hole circle (at 2.54 -20.32 90) (size 1.524 1.524) (drill 0.762) (layers *.Cu *.Mask F.SilkS))
+    (pad 2 thru_hole circle (at 2.54 -22.86 90) (size 1.524 1.524) (drill 0.762) (layers *.Cu *.Mask F.SilkS))
+    (pad 1 thru_hole circle (at 2.54 -25.4 90) (size 1.524 1.524) (drill 0.762) (layers *.Cu *.Mask F.SilkS))
+    (pad 10 thru_hole circle (at 2.54 -2.54 90) (size 1.524 1.524) (drill 0.762) (layers *.Cu *.Mask F.SilkS))
+    (pad 11 thru_hole circle (at 5.08 -2.54 90) (size 1.524 1.524) (drill 0.762) (layers *.Cu *.Mask F.SilkS))
+    (pad 12 thru_hole circle (at 7.62 -2.54 90) (size 1.524 1.524) (drill 0.762) (layers *.Cu *.Mask F.SilkS))
+    (pad 13 thru_hole circle (at 10.16 -2.54 90) (size 1.524 1.524) (drill 0.762) (layers *.Cu *.Mask F.SilkS))
     (pad 14 thru_hole circle (at 12.7 -2.54 90) (size 1.524 1.524) (drill 0.762) (layers *.Cu *.Mask F.SilkS))
-    (pad 13 thru_hole circle (at 15.24 -2.54 90) (size 1.524 1.524) (drill 0.762) (layers *.Cu *.Mask F.SilkS))
-    (pad 12 thru_hole circle (at 17.78 -2.54 90) (size 1.524 1.524) (drill 0.762) (layers *.Cu *.Mask F.SilkS))
-    (pad 11 thru_hole circle (at 20.32 -2.54 90) (size 1.524 1.524) (drill 0.762) (layers *.Cu *.Mask F.SilkS))
-    (pad 10 thru_hole circle (at 22.86 -2.54 90) (size 1.524 1.524) (drill 0.762) (layers *.Cu *.Mask F.SilkS))
-    (pad 9 thru_hole circle (at 22.86 -5.08 90) (size 1.524 1.524) (drill 0.762) (layers *.Cu *.Mask F.SilkS))
-    (pad 8 thru_hole circle (at 22.86 -7.62 90) (size 1.524 1.524) (drill 0.762) (layers *.Cu *.Mask F.SilkS))
-    (pad 7 thru_hole circle (at 22.86 -10.16 90) (size 1.524 1.524) (drill 0.762) (layers *.Cu *.Mask F.SilkS))
-    (pad 6 thru_hole circle (at 22.86 -12.7 90) (size 1.524 1.524) (drill 0.762) (layers *.Cu *.Mask F.SilkS))
-    (pad 5 thru_hole circle (at 22.86 -15.24 90) (size 1.524 1.524) (drill 0.762) (layers *.Cu *.Mask F.SilkS))
-    (pad 4 thru_hole circle (at 22.86 -17.78 90) (size 1.524 1.524) (drill 0.762) (layers *.Cu *.Mask F.SilkS))
-    (pad 3 thru_hole circle (at 22.86 -20.32 90) (size 1.524 1.524) (drill 0.762) (layers *.Cu *.Mask F.SilkS))
-    (pad 2 thru_hole circle (at 22.86 -22.86 90) (size 1.524 1.524) (drill 0.762) (layers *.Cu *.Mask F.SilkS))
-    (pad 1 thru_hole rect (at 22.86 -25.4 90) (size 1.524 1.524) (drill 0.762) (layers *.Cu *.Mask F.SilkS))
+    (pad 15 thru_hole circle (at 15.24 -2.54 90) (size 1.524 1.524) (drill 0.762) (layers *.Cu *.Mask F.SilkS))
+    (pad 16 thru_hole circle (at 17.78 -2.54 90) (size 1.524 1.524) (drill 0.762) (layers *.Cu *.Mask F.SilkS))
+    (pad 17 thru_hole circle (at 20.32 -2.54 90) (size 1.524 1.524) (drill 0.762) (layers *.Cu *.Mask F.SilkS))
+    (pad 18 thru_hole circle (at 22.86 -2.54 90) (size 1.524 1.524) (drill 0.762) (layers *.Cu *.Mask F.SilkS))
+    (pad 19 thru_hole circle (at 22.86 -5.08 90) (size 1.524 1.524) (drill 0.762) (layers *.Cu *.Mask F.SilkS))
+    (pad 20 thru_hole circle (at 22.86 -7.62 90) (size 1.524 1.524) (drill 0.762) (layers *.Cu *.Mask F.SilkS))
+    (pad 21 thru_hole circle (at 22.86 -10.16 90) (size 1.524 1.524) (drill 0.762) (layers *.Cu *.Mask F.SilkS))
+    (pad 22 thru_hole circle (at 22.86 -12.7 90) (size 1.524 1.524) (drill 0.762) (layers *.Cu *.Mask F.SilkS))
+    (pad 23 thru_hole circle (at 22.86 -15.24 90) (size 1.524 1.524) (drill 0.762) (layers *.Cu *.Mask F.SilkS))
+    (pad 24 thru_hole circle (at 22.86 -17.78 90) (size 1.524 1.524) (drill 0.762) (layers *.Cu *.Mask F.SilkS))
+    (pad 25 thru_hole circle (at 22.86 -20.32 90) (size 1.524 1.524) (drill 0.762) (layers *.Cu *.Mask F.SilkS))
+    (pad 26 thru_hole circle (at 22.86 -22.86 90) (size 1.524 1.524) (drill 0.762) (layers *.Cu *.Mask F.SilkS))
+    (pad 27 thru_hole rect (at 22.86 -25.4 90) (size 1.524 1.524) (drill 0.762) (layers *.Cu *.Mask F.SilkS))
   )
   (dimension 25.4 (width 0.3) (layer Dwgs.User)
