File: template/Arduino_Pro_Micro/Arduino-Pro-Micro.kicad_pcb (KiCad board)
At the start: 2 copper layers, 17.8 x 33 mm, 3 parts, among them J1 Digital, J2 Analog

Commit message: improved board drawings
Parts:
- removed REF**: USB_Micro-B, Connectors:USB_Micro-B
