File: template/Arduino_Pro_Micro/Arduino-Pro-Micro.sch (KiCad schematic (older format))
At the start: 2 parts, among them J1 Digital, J2 Analog

Commit message: improved board drawings
Changed lines of the file:
@@
 LIBS:contrib
 LIBS:valves
-LIBS:Arduino-Pro-Micro-cache
 EELAYER 25 0
 EELAYER END
@@
 Wire Wire Line
 	9450 1250 9450 2450
-Text Notes 9200 650  0    60   ~ 0
+Text Notes 9250 650  0    60   ~ 0
 Shield Arduino Pro Micro
 Wire Notes Line
